File: zx/pentagon 128 portable/469devboard/469devboard.sch (KiCad schematic (older format))
At the start: 10 parts, among them J1 Conn_02x17_Odd_Even, J2 Conn_ARM_JTAG_SWD_20, J3 Micro_SD_Card, U1 STM32F469IITx, Y1 NX3215SA-32.768K, Y2 NX3225GD-8.0M

Commit message: updated power lines
Parts:
- added BT1: cr1220 holder, symbol Device:Battery_Cell
- added C10, C12, C17, C19, C20, C21, C22, C23, C24, C25, C26, C27, C28, C29, C30, C31, C32, C33, C34, C35, C36, C37: 100nF, symbol Device:C_Small
- added C11, C16, C18: 1uF, symbol Device:CP_Small
- added C13, C6, C7: 2.2uF, symbol Device:C_Small
- added C14, C15: 4.7uF, symbol Device:CP_Small
- added C5: 100nF, Capacitor_SMD:C_0402_1005Metric, symbol Device:C_Small
- added C8, C9: 10uF, symbol Device:CP_Small
- added FB1: FCM1608KF-601T03, symbol Device:Ferrite_Bead_Small
- added J10: USB_B_Mini, symbol Connector:USB_B_Mini
- added J4: Conn_01x03_Male, Connector_PinHeader_2.54mm:PinHeader_1x03_P2.54mm_Vertical, symbol Connector:Conn_01x03_Male
- added J5, J6, J7, J8, J9: Conn_02x40_Counter_Clockwise, Connector_PinHeader_2.54mm:PinHeader_2x40_P2.54mm_Vertical, symbol Connector_Generic:Conn_02x40_Counter_Clockwise
- added R1: 10k, Resistor_SMD:R_0402_1005Metric, symbol Device:R_Small
- added R2, R5: 100k, Resistor_SMD:R_0402_1005Metric, symbol Device:R_Small
- added R3, R6, R7, R8: 10k, symbol Device:R_Small
- added R4: 0, symbol Device:R_Small
- added SW1: SW_Push, Button_Switch_SMD:SW_DIP_SPSTx01_Slide_6.7x4.1mm_W6.73mm_P2.54mm_LowProfile_JPin, symbol Switch:SW_Push
- added U2: LD1117S33TR_SOT223, Package_TO_SOT_SMD:SOT-223-3_TabPin2, symbol Regulator_Linear:LD1117S33TR_SOT223
Connections:
- net labels added: +5V, DSI_VDD12, VDD_A, VDD_MCU, VDD_REF+
- wire segments 210 -> 347
Other:
- note added: "Low ESR"

Commit message: upadted connectors
Parts:
- removed J5, J6, J7, J8: Conn_02x40_Counter_Clockwise, Connector_PinHeader_2.54mm:PinHeader_2x40_P2.54mm_Vertical, symbol Connector_Generic:Conn_02x40_Counter_Clockwise
- added J11: DSI, Connector_PinHeader_2.54mm:PinHeader_1x06_P2.54mm_Vertical, symbol Connector:Conn_01x06_Male
- added J5, J6, J7, J8: Conn_02x40_Odd_Even, Connector_PinHeader_2.54mm:PinHeader_2x40_P2.54mm_Vertical, symbol Connector_Generic:Conn_02x40_Odd_Even
- added R9: 10k, Resistor_SMD:R_0402_1005Metric, symbol Device:R_Small
- BT1: footprint (none) -> Battery:BatteryHolder_LINX_BAT-HLD-012-SMT
- C10, C11, C12, C13, C14, C15, C16, C17, C18, C19, C20, C21, C22, C23, C24, C25, C26, C27, C28, C29, C30, C31, C32, C33, C34, C35, C36, C37, C6, C7, C8, C9: footprint (none) -> Capacitor_SMD:C_0402_1005Metric
- J10: footprint (none) -> Connector_USB:USB_Mini-B_Lumberg_2486_01_Horizontal
- R3, R4, R6, R7, R8: footprint (none) -> Resistor_SMD:R_0402_1005Metric
Connections:
- net labels added: PA0, PA1, PA10, PA11, PA12, PA13, PA14, PA15, PA2, PA3, PA4, PA5, PA6, PA7, PA8, PA9, PB0, PB1, PB10, PB11, PB12, PB13, PB14, PB15, PB2, PB3, PB4, PB5, PB6, PB7, PB8, PB9, PC0, PC1, PC10, PC11, PC12, PC13, PC2, PC3, PC4, PC5, PC6, PC7, PC8, PC9, PD0, PD1, PD10, PD11, PD12, PD13, PD14, PD15, PD2, PD3, PD4, PD5, PD6, PD7, PD8, PD9, PE0, PE1, PE10, PE11, PE12, PE13, PE14, PE15, PE2, PE3, PE4, PE5, PE6, PE7, PE8, PE9, PF0, PF1, PF10, PF11, PF12, PF13, PF14, PF15, PF2, PF3, PF4, PF5, PF6, PF7, PF8, PF9, PG0, PG1, PG10, PG11, PG12, PG13, PG14, PG15, PG2, PG3, PG4, PG5, PG6, PG7, PG8, PG9, PH2, PH3, PH4, PH5, PH6, PH7, PI0, PI1, PI10, PI11, PI3, PI4, PI5, PI6, PI7, PI8, PI9
- wire segments 347 -> 353
Other:
- moved on the sheet: C1, C2, C3, C4, J3, J9, Y1, Y2

Commit message: update devboard routing
Parts:
- removed BT1: cr1220 holder, Battery:BatteryHolder_LINX_BAT-HLD-012-SMT, symbol Device:Battery_Cell
- removed J10: USB_B_Mini, Connector_USB:USB_Mini-B_Lumberg_2486_01_Horizontal, symbol Connector:USB_B_Mini
- removed J3: Micro_SD_Card, pentagon128:112JTDARR, symbol Connector:Micro_SD_Card
- removed J5, J6, J7, J8: Conn_02x40_Odd_Even, Connector_PinHeader_2.54mm:PinHeader_2x40_P2.54mm_Vertical, symbol Connector_Generic:Conn_02x40_Odd_Even
- removed J9: Conn_02x40_Counter_Clockwise, Connector_PinHeader_2.54mm:PinHeader_2x40_P2.54mm_Vertical, symbol Connector_Generic:Conn_02x40_Counter_Clockwise
- removed R4: 0, Resistor_SMD:R_0402_1005Metric, symbol Device:R_Small
- removed Y2: NX3225GD-8.0M, pentagon128:Crystal_SMD_3225-4Pin_3.2x2.5mm_HandSoldering, symbol Device:Crystal
- added C38, C39, C40, C41, C42, C43, C44, C45, C46, C47, C48, C49: 100nF, Capacitor_SMD:C_0402_1005Metric, symbol Device:C_Small
- added IC1: 1072, SamacSys_Parts:1072, symbol SamacSys_Parts:1072
- added J3: 10033526-N3212LF, SamacSys_Parts:10033526N3212LF, symbol SamacSys_Parts:10033526-N3212LF
- added J5: Conn_01x35_Male, Connector_PinHeader_2.54mm:PinHeader_1x35_P2.54mm_Vertical, symbol Connector:Conn_01x35_Male
- added J6: Conn_01x36_Male, Connector_PinHeader_2.54mm:PinHeader_1x36_P2.54mm_Vertical, symbol Connector:Conn_01x36_Male
- added J7: Conn_01x23_Male, Connector_PinHeader_2.54mm:PinHeader_1x23_P2.54mm_Vertical, symbol Connector:Conn_01x23_Male
- added J8: Conn_01x30_Male, Connector_PinHeader_2.54mm:PinHeader_1x30_P2.54mm_Vertical, symbol Connector:Conn_01x30_Male
- added J9: 104031-0811, SamacSys_Parts:1040310811, symbol SamacSys_Parts:104031-0811
- added R10: 220, Resistor_SMD:R_0402_1005Metric, symbol Device:R_Small
- added Y2: ABM3B-8.000MHZ-10-1-U-T, Crystal:Crystal_SMD_Abracon_ABM3B-4Pin_5.0x3.2mm, symbol Device:Crystal_GND24_Small
- C6, C7: footprint Capacitor_SMD:C_0402_1005Metric -> Capacitor_SMD:C_1210_3225Metric_Pad1.42x2.65mm_HandSolder
- FB1: value FCM1608KF-601T03 -> GZ2012D601TF; footprint (none) -> Capacitor_SMD:C_0805_2012Metric
- J2: footprint Connector_PinHeader_2.54mm:PinHeader_2x10_P2.54mm_Horizontal -> Connector_PinHeader_2.54mm:PinHeader_2x10_P2.54mm_Vertical
- Y1: value NX3215SA-32.768K -> Q13FC1350000400; footprint Crystal:Crystal_SMD_G8-2Pin_3.2x1.5mm_HandSoldering -> Crystal:Crystal_SMD_G8-2Pin_3.2x1.5mm
Connections:
- wire segments 353 -> 388
Other:
- moved on the sheet: R5
