File: zx/pentagon 128 portable/schematic/ZX Keyboard buttons/ZX Keyboard_buttons.kicad_pcb (KiCad board)
At the start: 2 copper layers, 99 x 66 mm, 51 parts, among them IC1 SN74LS245DW, IC2 SN74LS27N, IC3 SN74LS245DW, J1 Conn_01x03, J2 Conn_01x14, J3 Conn_01x02

Commit message: fixed keyboard
Parts:
- removed IC1, IC3: SN74LS245DW, SamacSys_Parts:SOIC127P1030X265-20N
- removed IC2: SN74LS27N, SamacSys_Parts:DIP794W53P254L1930H508Q14N
- removed J2: Conn_01x14, Connector_PinHeader_2.54mm:PinHeader_1x14_P2.54mm_Vertical
- removed J3: Conn_01x02, Connector_PinHeader_2.54mm:PinHeader_1x02_P2.54mm_Vertical
- removed R1, R2, R3, R4, R?-R1: 1.5K, Resistor_SMD:R_0402_1005Metric
- J1: value Conn_01x03 -> Conn_01x13; footprint Connector_PinHeader_2.54mm:PinHeader_1x03_P2.54mm_Vertical -> Connector_PinHeader_2.54mm:PinHeader_1x13_P2.54mm_Vertical
- moved J1 30.0 mm to (60.7, 99.1), turned to 90 degrees
Connections:
- J1 pad 1: /A0 -> /K_A8
- J1 pad 2: /~IORQ -> /K_A9
- J1 pad 3: /~RD -> /K_A10
Routing:
- net GND: track 89.2 -> 0.00 mm, vias 1 -> 0
- net +5V: track 49.7 -> 0.00 mm, vias 2 -> 0
- net /KEY_ENBL: track 29.3 -> 0.00 mm
- net /K_A8: track 114.2 -> 94.0 mm
- net /A14: track 19.7 -> 0.00 mm
- net /K_A9: track 108.4 -> 88.8 mm
- net /K_A10: track 103.1 -> 83.6 mm
- net /A13: track 19.2 -> 0.00 mm
- net /A12: track 18.6 -> 0.00 mm
- net /A11: track 18.1 -> 0.00 mm
- net /A8: track 18.1 -> 0.00 mm
- net /A10: track 17.6 -> 0.00 mm
- net /A15: track 17.3 -> 0.00 mm
- net /K_A15: track 131.5 -> 114.3 mm
- net /A9: track 17.1 -> 0.00 mm
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Other:
- board size 99 x 66 mm -> 99 x 46 mm
- board text added: "K_A10"
- board text added: "K_A11"
- board text added: "K_A12"
- board text added: "K_A13"
- board text added: "K_A14"
- board text added: "K_A15"
- board text added: "K_A8"
- board text added: "K_A9"
- board text added: "K_D0"
- board text added: "K_D1"
- board text added: "K_D2"
- board text added: "K_D3"
- board text added: "K_D4"
- board text removed: "+5V"
- board text removed: "A0"
- board text removed: "A10"
- board text removed: "A11"
- board text removed: "A12"
- board text removed: "A13"
- board text removed: "A14"
- board text removed: "A15"
- board text removed: "A8"
- board text removed: "A9"
- board text removed: "D0"
- board text removed: "D1"
- board text removed: "D2"
- board text removed: "D3"
- board text removed: "D4"
- board text removed: "GND"
- board text removed: "KEY_ENBL"
- board text removed: "~IORQ"
- board text removed: "~RD"

Commit message: added z80 pdip. updated all boards
Other:
- board text added: "JLCJLCJLCJLC"
