File: zx/pentagon 128 portable/schematic/ZX Keyboard logic/ZX Keyboard logic.sch (KiCad schematic (older format))
At the start: 51 parts, among them IC1 SN74LS245DW, IC2 SN74LS27N, IC3 SN74LS245DW, J1 Conn_01x03, J2 Conn_01x14, J3 Conn_01x02

Commit message: fixed keyboard
Parts:
- removed S1: 1, SamacSys_Parts:118259104, symbol SamacSys_Parts:1-1825910-4
- removed S10: 0, SamacSys_Parts:118259104, symbol SamacSys_Parts:1-1825910-4
- removed S11: Q, SamacSys_Parts:118259104, symbol SamacSys_Parts:1-1825910-4
- removed S12: W, SamacSys_Parts:118259104, symbol SamacSys_Parts:1-1825910-4
- removed S13: E, SamacSys_Parts:118259104, symbol SamacSys_Parts:1-1825910-4
- removed S14: R, SamacSys_Parts:118259104, symbol SamacSys_Parts:1-1825910-4
- removed S15: T, SamacSys_Parts:118259104, symbol SamacSys_Parts:1-1825910-4
- removed S16: Y, SamacSys_Parts:118259104, symbol SamacSys_Parts:1-1825910-4
- removed S17: U, SamacSys_Parts:118259104, symbol SamacSys_Parts:1-1825910-4
- removed S18: I, SamacSys_Parts:118259104, symbol SamacSys_Parts:1-1825910-4
- removed S19: O, SamacSys_Parts:118259104, symbol SamacSys_Parts:1-1825910-4
- removed S2: 2, SamacSys_Parts:118259104, symbol SamacSys_Parts:1-1825910-4
- removed S20: P, SamacSys_Parts:118259104, symbol SamacSys_Parts:1-1825910-4
- removed S21: A, SamacSys_Parts:118259104, symbol SamacSys_Parts:1-1825910-4
- removed S22: S, SamacSys_Parts:118259104, symbol SamacSys_Parts:1-1825910-4
- removed S23: D, SamacSys_Parts:118259104, symbol SamacSys_Parts:1-1825910-4
- removed S24: F, SamacSys_Parts:118259104, symbol SamacSys_Parts:1-1825910-4
- removed S25: G, SamacSys_Parts:118259104, symbol SamacSys_Parts:1-1825910-4
- removed S26: H, SamacSys_Parts:118259104, symbol SamacSys_Parts:1-1825910-4
- removed S27: J, SamacSys_Parts:118259104, symbol SamacSys_Parts:1-1825910-4
- removed S28: K, SamacSys_Parts:118259104, symbol SamacSys_Parts:1-1825910-4
- removed S29: L, SamacSys_Parts:118259104, symbol SamacSys_Parts:1-1825910-4
- removed S3: 3, SamacSys_Parts:118259104, symbol SamacSys_Parts:1-1825910-4
- removed S30: ENTER, SamacSys_Parts:118259104, symbol SamacSys_Parts:1-1825910-4
- removed S31: CAPS, SamacSys_Parts:118259104, symbol SamacSys_Parts:1-1825910-4
- removed S32: Z, SamacSys_Parts:118259104, symbol SamacSys_Parts:1-1825910-4
- removed S33: X, SamacSys_Parts:118259104, symbol SamacSys_Parts:1-1825910-4
- removed S34: C, SamacSys_Parts:118259104, symbol SamacSys_Parts:1-1825910-4
- removed S35: V, SamacSys_Parts:118259104, symbol SamacSys_Parts:1-1825910-4
- removed S36: B, SamacSys_Parts:118259104, symbol SamacSys_Parts:1-1825910-4
- removed S37: N, SamacSys_Parts:118259104, symbol SamacSys_Parts:1-1825910-4
- removed S38: M, SamacSys_Parts:118259104, symbol SamacSys_Parts:1-1825910-4
- removed S39: SYMB, SamacSys_Parts:118259104, symbol SamacSys_Parts:1-1825910-4
- removed S4: 4, SamacSys_Parts:118259104, symbol SamacSys_Parts:1-1825910-4
- removed S40: SPACE, SamacSys_Parts:118259104, symbol SamacSys_Parts:1-1825910-4
- removed S5: 5, SamacSys_Parts:118259104, symbol SamacSys_Parts:1-1825910-4
- removed S6: 6, SamacSys_Parts:118259104, symbol SamacSys_Parts:1-1825910-4
- removed S7: 7, SamacSys_Parts:118259104, symbol SamacSys_Parts:1-1825910-4
- removed S8: 8, SamacSys_Parts:118259104, symbol SamacSys_Parts:1-1825910-4
- removed S9: 9, SamacSys_Parts:118259104, symbol SamacSys_Parts:1-1825910-4
- added J4: Conn_01x13, Connector_PinSocket_2.54mm:PinSocket_1x13_P2.54mm_Vertical, symbol Connector_Generic:Conn_01x13
Connections:
- wire segments 266 -> 79
