File: zx/pentagon 128 portable/schematic/RAM_ROM_devboard 128K/RAM_ROM_devboard.sch (KiCad schematic (older format))
At the start: 9 parts, among them IC1 IS62C1024AL-35QLI, IC2 SN74AHCT04D, J1 Conn_02x14_Odd_Even, J2 8432-11B1-RK-TP, J3 Conn_02x08_Odd_Even, J4 Conn_02x04_Odd_Even, J5 Conn_02x06_Odd_Even, J6 Conn_02x06_Odd_Even

Commit message: updated ram 128k, 512k, keyboard
Parts:
- removed C1: C_Small, Capacitor_SMD:C_0402_1005Metric, symbol Device:C_Small
- removed IC2: SN74AHCT04D, SamacSys_Parts:SOIC127P600X175-14N, symbol SamacSys_Parts:SN74AHCT04D
Connections:
- wire segments 157 -> 145
Changed lines of the file:
@@
 Wire Wire Line
 	4700 5300 5150 5300
-$Comp
-L SamacSys_Parts:SN74AHCT04D IC2
-U 1 1 5F614487
-P 6000 1550
-F 0 "IC2" H 6500 1815 50  0000 C CNN
-F 1 "SN74AHCT04D" H 6500 1724 50  0000 C CNN
-F 2 "SamacSys_Parts:SOIC127P600X175-14N" H 6850 1650 50  0001 L CNN
-F 3 "http://www.ti.com/lit/gpn/SN74AHCT04" H 6850 1550 50  0001 L CNN
-F 4 "IC, HEX INVERTER, SMD" H 6850 1450 50  0001 L CNN "Description"
-F 5 "1.75" H 6850 1350 50  0001 L CNN "Height"
-F 6 "595-SN74AHCT04D" H 6850 1250 50  0001 L CNN "Mouser Part Number"
-F 7 "https://www.mouser.co.uk/ProductDetail/Texas-Instruments/SN74AHCT04D?qs=bkMXpVdiF42hAjN5593l5w%3D%3D" H 6850 1150 50  0001 L CNN "Mouser Price/Stock"
-F 8 "Texas Instruments" H 6850 1050 50  0001 L CNN "Manufacturer_Name"
-F 9 "SN74AHCT04D" H 6850 950 50  0001 L CNN "Manufacturer_Part_Number"
-	1    6000 1550
-	1    0    0    -1
-$EndComp
-Wire Wire Line
-	6000 1550 5650 1550
-Wire Wire Line
-	6000 1650 5650 1650
-Text Label 5650 1550 0    50   ~ 0
-~RAM_CE
-Text Label 5650 1650 0    50   ~ 0
-RAM_CE
 Wire Wire Line
 	4800 1550 5200 1550
 Wire Wire Line
 	4800 1650 5200 1650
-Wire Wire Line
-	4800 1750 5200 1750
 Wire Wire Line
 	4800 1850 5200 1850
@@
 $EndComp
 $Comp
-L power:+5V #PWR0104
-U 1 1 5F645708
-P 7050 1450
-F 0 "#PWR0104" H 7050 1300 50  0001 C CNN
-F 1 "+5V" H 7065 1623 50  0000 C CNN
-F 2 "" H 7050 1450 50  0001 C CNN
-F 3 "" H 7050 1450 50  0001 C CNN
-	1    7050 1450
-	1    0    0    -1
-$EndComp
-$Comp
-L power:GND #PWR0105
-U 1 1 5F648D11
-P 5900 2250
-F 0 "#PWR0105" H 5900 2000 50  0001 C CNN
-F 1 "GND" H 5905 2077 50  0000 C CNN
-F 2 "" H 5900 2250 50  0001 C CNN
-F 3 "" H 5900 2250 50  0001 C CNN
-	1    5900 2250
-	1    0    0    -1
-$EndComp
-Wire Wire Line
-	7000 1550 7050 1550
-Wire Wire Line
-	7050 1550 7050 1450
-Wire Wire Line
-	6000 2150 5900 2150
-Wire Wire Line
-	5900 2150 5900 2250
-$Comp
 L power:GND #PWR0106
 U 1 1 5F64E1DA
@@
 Text Label 1700 5550 0    50   ~ 0
 RAM_A16
+Text Label 1700 5750 0    50   ~ 0
+~RAM_OE
 Text Label 1700 5650 0    50   ~ 0
-~RAM_OE
-Text Label 1700 5750 0    50   ~ 0
 ~RAM_CE
 Text Label 1700 5850 0    50   ~ 0
@@
 Text Label 650  5850 0    50   ~ 0
 ~RAM_WE
+Text Label 650  5650 0    50   ~ 0
+~RAM_CE
 Text Label 650  5750 0    50   ~ 0
-~RAM_CE
-Text Label 650  5650 0    50   ~ 0
 ~RAM_OE
 Text Label 650  5350 0    50   ~ 0
@@
 	6050 4400 6050 4300
 Connection ~ 6050 4400
-$Comp
-L power:+5V #PWR0109
-U 1 1 5F62EBF2
-P 5850 1750
-F 0 "#PWR0109" H 5850 1600 50  0001 C CNN
-F 1 "+5V" H 5865 1923 50  0000 C CNN
-F 2 "" H 5850 1750 50  0001 C CNN
-F 3 "" H 5850 1750 50  0001 C CNN
-	1    5850 1750
-	0    -1   -1   0
-$EndComp
-$Comp
-L power:+5V #PWR0110
-U 1 1 5F62F7B9
-P 5850 1950
-F 0 "#PWR0110" H 5850 1800 50  0001 C CNN
-F 1 "+5V" H 5865 2123 50  0000 C CNN
-F 2 "" H 5850 1950 50  0001 C CNN
-F 3 "" H 5850 1950 50  0001 C CNN
-	1    5850 1950
-	0    -1   -1   0
-$EndComp
-Wire Wire Line
-	6000 1950 5850 1950
-Wire Wire Line
-	6000 1750 5850 1750
-$Comp
-L power:+5V #PWR0111
-U 1 1 5F647A6C
-P 7100 1850
-F 0 "#PWR0111" H 7100 1700 50  0001 C CNN
-F 1 "+5V" H 7115 2023 50  0000 C CNN
-F 2 "" H 7100 1850 50  0001 C CNN
-F 3 "" H 7100 1850 50  0001 C CNN
-	1    7100 1850
-	0    1    1    0
-$EndComp
-$Comp
-L power:+5V #PWR0112
-U 1 1 5F6486F7
-P 7100 2050
-F 0 "#PWR0112" H 7100 1900 50  0001 C CNN
-F 1 "+5V" H 7115 2223 50  0000 C CNN
-F 2 "" H 7100 2050 50  0001 C CNN
-F 3 "" H 7100 2050 50  0001 C CNN
-	1    7100 2050
-	0    1    1    0
-$EndComp
-Wire Wire Line
-	7000 1650 7000 1550
-Connection ~ 7000 1550
-Wire Wire Line
-	7000 1850 7100 1850
-Wire Wire Line
-	7000 2050 7100 2050
-$Comp
-L Device:C_Small C1
-U 1 1 5F66D823
-P 6450 2600
-F 0 "C1" V 6221 2600 50  0000 C CNN
-F 1 "C_Small" V 6312 2600 50  0000 C CNN
-F 2 "Capacitor_SMD:C_0402_1005Metric" H 6450 2600 50  0001 C CNN
-F 3 "~" H 6450 2600 50  0001 C CNN
-	1    6450 2600
-	0    1    1    0
-$EndComp
-$Comp
-L power:GND #PWR0113
-U 1 1 5F66F725
-P 6250 2700
-F 0 "#PWR0113" H 6250 2450 50  0001 C CNN
-F 1 "GND" H 6255 2527 50  0000 C CNN
-F 2 "" H 6250 2700 50  0001 C CNN
-F 3 "" H 6250 2700 50  0001 C CNN
-	1    6250 2700
-	1    0    0    -1
-$EndComp
-$Comp
-L power:+5V #PWR0114
-U 1 1 5F670043
-P 6750 2600
-F 0 "#PWR0114" H 6750 2450 50  0001 C CNN
-F 1 "+5V" H 6765 2773 50  0000 C CNN
-F 2 "" H 6750 2600 50  0001 C CNN
-F 3 "" H 6750 2600 50  0001 C CNN
-	1    6750 2600
-	1    0    0    -1
-$EndComp
-Wire Wire Line
-	6550 2600 6750 2600
-Wire Wire Line
-	6350 2600 6250 2600
-Wire Wire Line
-	6250 2600 6250 2700
+Wire Wire Line
+	5350 1750 5350 1550
+Wire Wire Line
+	5350 1550 5200 1550
+Wire Wire Line
+	4800 1750 5350 1750
+Connection ~ 5200 1550
 $EndSCHEMATC
