File: zx/pentagon 128 portable/schematic/Pentagon128 portable/STM32.sch (KiCad schematic (older format))
At the start: 18 parts

Commit message: reorganizing. finished ram and keyboard, updated z80
Parts:
- removed C?: 104, symbol Device:C
- removed C? (x3): 106, symbol Device:C
- removed C? (x3): 22p, symbol Device:C
- removed IC? (x3): TXB0108PWR, SOP65P640X120-20N, symbol SamacSys_Parts:TXB0108PWR
- removed J?: LCD, symbol Connector_Generic_MountingPin:Conn_02x16_Odd_Even_MountingPin
- removed R? (x2): 1M, symbol Device:R
- removed R?: R, symbol Device:R
- removed SW?: SW_DIP_x01, symbol Switch:SW_DIP_x01
- removed U?: STM32F469IITx, Package_QFP:LQFP-176_24x24mm_P0.5mm, symbol MCU_ST_STM32F4:STM32F469IITx
- removed U?: STM32F407VETx, Package_QFP:LQFP-100_14x14mm_P0.5mm, symbol MCU_ST_STM32F4:STM32F407VETx
- removed Y?: 8M, symbol Device:Crystal
- added C1, C2: 3.0pF, Capacitor_SMD:C_0402_1005Metric, symbol Device:C_Small
- added C10, C12, C17, C19, C20, C21, C22, C23, C24, C25, C26, C27, C28, C29, C30, C31, C32, C33, C34, C35, C36, C37, C38, C39, C40, C41, C42, C43, C44, C45, C46, C47, C48, C49, C5: 100nF, Capacitor_SMD:C_0402_1005Metric, symbol Device:C_Small
- added C11, C16, C18: 1uF, Capacitor_SMD:C_0402_1005Metric, symbol Device:CP_Small
- added C13: 2.2uF, Capacitor_SMD:C_0402_1005Metric, symbol Device:C_Small
- added C14, C15: 4.7uF, Capacitor_SMD:C_0402_1005Metric, symbol Device:CP_Small
- added C3, C4: 8.2pF, Capacitor_SMD:C_0402_1005Metric, symbol Device:C_Small
- added C6, C7: 2.2uF, Capacitor_SMD:C_1210_3225Metric_Pad1.42x2.65mm_HandSolder, symbol Device:C_Small
- added C8, C9: 10uF, Capacitor_SMD:C_0402_1005Metric, symbol Device:CP_Small
- added FB1: GZ2012D601TF, Capacitor_SMD:C_0805_2012Metric, symbol Device:Ferrite_Bead_Small
- added IC1: 1072, SamacSys_Parts:1072, symbol SamacSys_Parts:1072
- added J1: Conn_02x17_Odd_Even, Connector_PinSocket_2.54mm:PinSocket_2x17_P2.54mm_Vertical, symbol Connector_Generic:Conn_02x17_Odd_Even
- added J11: DSI, Connector_PinHeader_2.54mm:PinHeader_1x06_P2.54mm_Vertical, symbol Connector:Conn_01x06_Male
- added J2: Conn_ARM_JTAG_SWD_20, Connector_PinHeader_2.54mm:PinHeader_2x10_P2.54mm_Vertical, symbol Connector:Conn_ARM_JTAG_SWD_20
- added J3: 10033526-N3212LF, SamacSys_Parts:10033526N3212LF, symbol SamacSys_Parts:10033526-N3212LF
- added J4: Conn_01x03_Male, Connector_PinHeader_2.54mm:PinHeader_1x03_P2.54mm_Vertical, symbol Connector:Conn_01x03_Male
- added J9: 104031-0811, SamacSys_Parts:1040310811, symbol SamacSys_Parts:104031-0811
- added R1, R3, R6, R7, R8, R9: 10k, Resistor_SMD:R_0402_1005Metric, symbol Device:R_Small
- added R10: 220, Resistor_SMD:R_0402_1005Metric, symbol Device:R_Small
- added R2, R5: 100k, Resistor_SMD:R_0402_1005Metric, symbol Device:R_Small
- added SW1: SW_Push, Button_Switch_SMD:SW_DIP_SPSTx01_Slide_6.7x4.1mm_W6.73mm_P2.54mm_LowProfile_JPin, symbol Switch:SW_Push
- added U1: STM32F469IITx, Package_QFP:LQFP-176_24x24mm_P0.5mm, symbol MCU_ST_STM32F4:STM32F469IITx
- added U2: LD1117S33TR_SOT223, Package_TO_SOT_SMD:SOT-223-3_TabPin2, symbol Regulator_Linear:LD1117S33TR_SOT223
- added Y1: Q13FC1350000400, Crystal:Crystal_SMD_G8-2Pin_3.2x1.5mm, symbol Device:Crystal
- added Y2: ABM3B-8.000MHZ-10-1-U-T, Crystal:Crystal_SMD_Abracon_ABM3B-4Pin_5.0x3.2mm, symbol Device:Crystal_GND24_Small
Connections:
- net labels added: +3.3, +5V, DAC_OUT, DSI_VDD12, FMC_A16, FMC_D0, FMC_D1, FMC_D10, FMC_D11, FMC_D12, FMC_D13, FMC_D14, FMC_D15, FMC_D2, FMC_D3, FMC_D4, FMC_D5, FMC_D6, FMC_D7, FMC_D8, FMC_D9, FMC_NE1, FMC_NOE, FMC_NWE, HSE_IN, HSE_OUT, LSE_IN, LSE_OUT, NRST, PA0, PA1, PA10, PA11, PA12, PA13, PA14, PA15, PA2, PA3, PA4, PA5, PA6, PA7, PA8, PA9, PB0, PB1, PB10, PB11, PB12, PB13, PB14, PB15, PB2, PB3, PB4, PB5, PB6, PB7, PB8, PB9, PC0, PC1, PC10, PC11, PC12, PC13, PC2, PC3, PC4, PC5, PC6, PC7, PC8, PC9, PD0, PD1, PD10, PD11, PD12, PD13, PD14, PD15, PD2, PD3, PD4, PD5, PD6, PD7, PD8, PD9, PE0, PE1, PE10, PE11, PE12, PE13, PE14, PE15, PE2, PE3, PE4, PE5, PE6, PE7, PE8, PE9, PEN, PF0, PF1, PF10, PF11, PF12, PF13, PF14, PF15, PF2, PF3, PF4, PF5, PF6, PF7, PF8, PF9, PG0, PG1, PG10, PG11, PG12, PG13, PG14, PG15, PG2, PG3, PG4, PG5, PG6, PG7, PG8, PG9, PH2, PH3, PH4, PH5, PH6, PH7, PI0, PI1, PI10, PI11, PI3, PI4, PI5, PI6, PI7, PI8, PI9, SCIO_CMD, SCREEN_RESET, SDIO_CK, SYS_JTCK_SWCLK, SYS_JTDO_SWO, SYS_JTFO_SWO, SYS_JTMS_SWDIO, T_CLK, VDD_A, VDD_MCU, VDD_REF+
- net labels removed: AY_CLK, CPU_CLK, FSMC_A18, FSMC_A23, FSMC_D0, FSMC_D1, FSMC_D10, FSMC_D11, FSMC_D12, FSMC_D13, FSMC_D14, FSMC_D15, FSMC_D2, FSMC_D3, FSMC_D4, FSMC_D5, FSMC_D6, FSMC_D7, FSMC_D8, FSMC_D9, FSMC_NE1, FSMC_NOE, FSMC_NWE, JTMS_SWCLK, JTMS_SWDIO, JTMS_SWO, LCD_BL, OSC_IN, OSC_OUT, SDIO_SCK, STM_RESET, TAPE_IN, T_CS, T_SCK
- wire segments 116 -> 388
Other:
- note added: "Low ESR"

Commit message: some reordering in the main project
Parts:
- removed C1, C2: 3.0pF, Capacitor_SMD:C_0402_1005Metric, symbol Device:C_Small
- removed C10, C12, C17, C19, C20, C21, C22, C23, C24, C25, C26, C27, C28, C29, C30, C31, C32, C33, C34, C35, C36, C37, C38, C39, C40, C41, C42, C43, C44, C45, C46, C47, C48, C49, C5: 100nF, Capacitor_SMD:C_0402_1005Metric, symbol Device:C_Small
- removed C11, C16, C18: 1uF, Capacitor_SMD:C_0402_1005Metric, symbol Device:CP_Small
- removed C13: 2.2uF, Capacitor_SMD:C_0402_1005Metric, symbol Device:C_Small
- removed C14, C15: 4.7uF, Capacitor_SMD:C_0402_1005Metric, symbol Device:CP_Small
- removed C3, C4: 8.2pF, Capacitor_SMD:C_0402_1005Metric, symbol Device:C_Small
- removed C6, C7: 2.2uF, Capacitor_SMD:C_1210_3225Metric_Pad1.42x2.65mm_HandSolder, symbol Device:C_Small
- removed C8, C9: 10uF, Capacitor_SMD:C_0402_1005Metric, symbol Device:CP_Small
- removed FB1: GZ2012D601TF, Capacitor_SMD:C_0805_2012Metric, symbol Device:Ferrite_Bead_Small
- removed IC1: 1072, SamacSys_Parts:1072, symbol SamacSys_Parts:1072
- removed J1: Conn_02x17_Odd_Even, Connector_PinSocket_2.54mm:PinSocket_2x17_P2.54mm_Vertical, symbol Connector_Generic:Conn_02x17_Odd_Even
- removed J11: DSI, Connector_PinHeader_2.54mm:PinHeader_1x06_P2.54mm_Vertical, symbol Connector:Conn_01x06_Male
- removed J2: Conn_ARM_JTAG_SWD_20, Connector_PinHeader_2.54mm:PinHeader_2x10_P2.54mm_Vertical, symbol Connector:Conn_ARM_JTAG_SWD_20
- removed J3: 10033526-N3212LF, SamacSys_Parts:10033526N3212LF, symbol SamacSys_Parts:10033526-N3212LF
- removed J4: Conn_01x03_Male, Connector_PinHeader_2.54mm:PinHeader_1x03_P2.54mm_Vertical, symbol Connector:Conn_01x03_Male
- removed J9: 104031-0811, SamacSys_Parts:1040310811, symbol SamacSys_Parts:104031-0811
- removed R1, R3, R6, R7, R8, R9: 10k, Resistor_SMD:R_0402_1005Metric, symbol Device:R_Small
- removed R10: 220, Resistor_SMD:R_0402_1005Metric, symbol Device:R_Small
- removed R2, R5: 100k, Resistor_SMD:R_0402_1005Metric, symbol Device:R_Small
- removed SW1: SW_Push, Button_Switch_SMD:SW_DIP_SPSTx01_Slide_6.7x4.1mm_W6.73mm_P2.54mm_LowProfile_JPin, symbol Switch:SW_Push
- removed U1: STM32F469IITx, Package_QFP:LQFP-176_24x24mm_P0.5mm, symbol MCU_ST_STM32F4:STM32F469IITx
- removed U2: LD1117S33TR_SOT223, Package_TO_SOT_SMD:SOT-223-3_TabPin2, symbol Regulator_Linear:LD1117S33TR_SOT223
- removed Y1: Q13FC1350000400, Crystal:Crystal_SMD_G8-2Pin_3.2x1.5mm, symbol Device:Crystal
- removed Y2: ABM3B-8.000MHZ-10-1-U-T, Crystal:Crystal_SMD_Abracon_ABM3B-4Pin_5.0x3.2mm, symbol Device:Crystal_GND24_Small
Connections:
- net labels removed: +3.3, +3.3V, +5V, DAC_OUT, DSI_VDD12, FMC_A16, FMC_D0, FMC_D1, FMC_D10, FMC_D11, FMC_D12, FMC_D13, FMC_D14, FMC_D15, FMC_D2, FMC_D3, FMC_D4, FMC_D5, FMC_D6, FMC_D7, FMC_D8, FMC_D9, FMC_NE1, FMC_NOE, FMC_NWE, GND, HSE_IN, HSE_OUT, LSE_IN, LSE_OUT, NRST, PA0, PA1, PA10, PA11, PA12, PA13, PA14, PA15, PA2, PA3, PA4, PA5, PA6, PA7, PA8, PA9, PB0, PB1, PB10, PB11, PB12, PB13, PB14, PB15, PB2, PB3, PB4, PB5, PB6, PB7, PB8, PB9, PC0, PC1, PC10, PC11, PC12, PC13, PC2, PC3, PC4, PC5, PC6, PC7, PC8, PC9, PD0, PD1, PD10, PD11, PD12, PD13, PD14, PD15, PD2, PD3, PD4, PD5, PD6, PD7, PD8, PD9, PE0, PE1, PE10, PE11, PE12, PE13, PE14, PE15, PE2, PE3, PE4, PE5, PE6, PE7, PE8, PE9, PEN, PF0, PF1, PF10, PF11, PF12, PF13, PF14, PF15, PF2, PF3, PF4, PF5, PF6, PF7, PF8, PF9, PG0, PG1, PG10, PG11, PG12, PG13, PG14, PG15, PG2, PG3, PG4, PG5, PG6, PG7, PG8, PG9, PH2, PH3, PH4, PH5, PH6, PH7, PI0, PI1, PI10, PI11, PI3, PI4, PI5, PI6, PI7, PI8, PI9, SCIO_CMD, SCREEN_RESET, SDIO_CK, SDIO_CMD, SDIO_D0, SDIO_D1, SDIO_D2, SDIO_D3, SYS_JTCK_SWCLK, SYS_JTDO_SWO, SYS_JTFO_SWO, SYS_JTMS_SWDIO, T_CLK, T_MISO, T_MOSI, VDD_A, VDD_MCU, VDD_REF+
- wire segments 388 -> 0
Other:
- note removed: "Low ESR"

Commit message: updated schemes
Changed lines of the file:
@@
 $EndDescr
 $Sheet
-S 9500 1150 1950 5300
+S 1900 1050 1950 5300
 U 5F7467A7
 F0 "stm32_cpu" 50
@@
 $EndSheet
 $Sheet
-S 12350 1300 1900 2700
+S 4750 1200 1900 2700
 U 5F747225
 F0 "stm32_power" 50
@@
 $EndSheet
 $Sheet
-S 9950 7800 850  1800
+S 2350 7700 850  1800
 U 5F8C0463
 F0 "stm32_crystall" 50
@@
 $EndSheet
 $Sheet
-S 11800 7450 1200 2150
+S 4200 7350 1200 2150
 U 5F98BCEA
 F0 "stm32_debug" 50
