File: zx/pentagon 128 portable/schematic/Pentagon128 portable/AY.sch (KiCad schematic (older format))
At the start: 11 parts

Commit message: updated schemes
Parts:
- C57, C58: renamed from C?; value 10.0 -> 10.0uF
- R16, R17: renamed from R?; value 4.7K -> 4.7k; footprint (none) -> Resistor_SMD:R_0402_1005Metric
- R18, R23: renamed from R?; value 5.1K -> 5.1k; footprint (none) -> Resistor_SMD:R_0402_1005Metric
- R19, R20: renamed from R?; value 1K -> 1k; footprint (none) -> Resistor_SMD:R_0402_1005Metric
- R21, R22: renamed from R?; value 2K -> 2k; footprint (none) -> Resistor_SMD:R_0402_1005Metric
- gave numbers to parts that had none: 1
Changed lines of the file:
@@
 $Descr A4 11693 8268
 encoding utf-8
-Sheet 4 14
+Sheet 8 14
 Title ""
 Date ""
@@
 $EndDescr
 $Comp
-L Audio:YM2149 U?
+L Audio:YM2149 U2
 U 1 1 5F5BE3B6
 P 3350 3500
-F 0 "U?" H 3350 4881 50  0000 C CNN
+F 0 "U2" H 3350 4881 50  0000 C CNN
 F 1 "YM2149" H 3350 4790 50  0000 C CNN
 F 2 "Package_DIP:DIP-40_W15.24mm" H 4000 2100 50  0001 C CNN
@@
 	2850 3200 2500 3200
 $Comp
-L power:+5V #PWR?
+L power:+5V #PWR039
 U 1 1 5F5C0B75
 P 2000 3800
-F 0 "#PWR?" H 2000 3650 50  0001 C CNN
+F 0 "#PWR039" H 2000 3650 50  0001 C CNN
 F 1 "+5V" V 2015 3928 50  0000 L CNN
 F 2 "" H 2000 3800 50  0001 C CNN
@@
 	2850 3400 2000 3400
 $Comp
-L power:+5V #PWR?
+L power:+5V #PWR037
 U 1 1 5F5C1A92
 P 2000 3400
-F 0 "#PWR?" H 2000 3250 50  0001 C CNN
+F 0 "#PWR037" H 2000 3250 50  0001 C CNN
 F 1 "+5V" H 2015 3573 50  0000 C CNN
 F 2 "" H 2000 3400 50  0001 C CNN
@@
 $EndComp
 $Comp
-L power:GND #PWR?
+L power:GND #PWR038
 U 1 1 5F5C1DB3
 P 2000 3500
-F 0 "#PWR?" H 2000 3250 50  0001 C CNN
+F 0 "#PWR038" H 2000 3250 50  0001 C CNN
 F 1 "GND" H 2005 3327 50  0000 C CNN
 F 2 "" H 2000 3500 50  0001 C CNN
@@
 	2850 3500 2000 3500
 $Comp
-L power:GND #PWR?
+L power:GND #PWR040
 U 1 1 5F5C263B
 P 3350 4850
-F 0 "#PWR?" H 3350 4600 50  0001 C CNN
+F 0 "#PWR040" H 3350 4600 50  0001 C CNN
 F 1 "GND" H 3355 4677 50  0000 C CNN
 F 2 "" H 3350 4850 50  0001 C CNN
@@
 $EndComp
 $Comp
-L power:+5V #PWR?
+L power:+5V #PWR035
 U 1 1 5F5C2C20
 P 3750 2100
-F 0 "#PWR?" H 3750 1950 50  0001 C CNN
+F 0 "#PWR035" H 3750 1950 50  0001 C CNN
 F 1 "+5V" H 3765 2273 50  0000 C CNN
 F 2 "" H 3750 2100 50  0001 C CNN
@@
 	3350 4700 3350 4850
 $Comp
-L Device:R R?
+L Device:R R16
 U 1 1 5F5C365A
 P 5500 1850
-F 0 "R?" H 5570 1896 50  0000 L CNN
-F 1 "4.7K" H 5570 1805 50  0000 L CNN
-F 2 "" V 5430 1850 50  0001 C CNN
+F 0 "R16" H 5570 1896 50  0000 L CNN
+F 1 "4.7k" H 5570 1805 50  0000 L CNN
+F 2 "Resistor_SMD:R_0402_1005Metric" V 5430 1850 50  0001 C CNN
 F 3 "~" H 5500 1850 50  0001 C CNN
 	1    5500 1850
@@
 $EndComp
 $Comp
-L Device:R R?
+L Device:R R17
 U 1 1 5F5C4183
 P 5850 1850
-F 0 "R?" H 5920 1896 50  0000 L CNN
-F 1 "4.7K" H 5920 1805 50  0000 L CNN
-F 2 "" V 5780 1850 50  0001 C CNN
+F 0 "R17" H 5920 1896 50  0000 L CNN
+F 1 "4.7k" H 5920 1805 50  0000 L CNN
+F 2 "Resistor_SMD:R_0402_1005Metric" V 5780 1850 50  0001 C CNN
 F 3 "~" H 5850 1850 50  0001 C CNN
 	1    5850 1850
@@
 $EndComp
 $Comp
-L Device:R R?
+L Device:R R21
 U 1 1 5F5C440C
 P 5500 2900
-F 0 "R?" H 5570 2946 50  0000 L CNN
-F 1 "2K" H 5570 2855 50  0000 L CNN
-F 2 "" V 5430 2900 50  0001 C CNN
+F 0 "R21" H 5570 2946 50  0000 L CNN
+F 1 "2k" H 5570 2855 50  0000 L CNN
+F 2 "Resistor_SMD:R_0402_1005Metric" V 5430 2900 50  0001 C CNN
 F 3 "~" H 5500 2900 50  0001 C CNN
 	1    5500 2900
@@
 $EndComp
 $Comp
-L Device:R R?
-U 1 1 5F5C4893
-P 5850 2900
-F 0 "R?" H 5920 2946 50  0000 L CNN
-F 1 "2K" H 5920 2855 50  0000 L CNN
-F 2 "" V 5780 2900 50  0001 C CNN
-F 3 "~" H 5850 2900 50  0001 C CNN
-	1    5850 2900
-	1    0    0    -1
-$EndComp
-$Comp
-L Device:R R?
+L Device:R R23
 U 1 1 5F5C4CDD
 P 6900 2900
-F 0 "R?" H 6970 2946 50  0000 L CNN
-F 1 "5.1K" H 6970 2855 50  0000 L CNN
-F 2 "" V 6830 2900 50  0001 C CNN
+F 0 "R23" H 6970 2946 50  0000 L CNN
+F 1 "5.1k" H 6970 2855 50  0000 L CNN
+F 2 "Resistor_SMD:R_0402_1005Metric" V 6830 2900 50  0001 C CNN
 F 3 "~" H 6900 2900 50  0001 C CNN
 	1    6900 2900
@@
 $EndComp
 $Comp
-L Device:R R?
+L Device:R R18
 U 1 1 5F5C4FC7
 P 6850 1850
-F 0 "R?" H 6920 1896 50  0000 L CNN
-F 1 "5.1K" H 6920 1805 50  0000 L CNN
-F 2 "" V 6780 1850 50  0001 C CNN
+F 0 "R18" H 6920 1896 50  0000 L CNN
+F 1 "5.1k" H 6920 1805 50  0000 L CNN
+F 2 "Resistor_SMD:R_0402_1005Metric" V 6780 1850 50  0001 C CNN
 F 3 "~" H 6850 1850 50  0001 C CNN
 	1    6850 1850
@@
 $EndComp
 $Comp
-L Device:R R?
+L Device:R R19
 U 1 1 5F5C547E
 P 4950 2150
-F 0 "R?" V 4743 2150 50  0000 C CNN
-F 1 "1K" V 4834 2150 50  0000 C CNN
-F 2 "" V 4880 2150 50  0001 C CNN
+F 0 "R19" V 4743 2150 50  0000 C CNN
+F 1 "1k" V 4834 2150 50  0000 C CNN
+F 2 "Resistor_SMD:R_0402_1005Metric" V 4880 2150 50  0001 C CNN
 F 3 "~" H 4950 2150 50  0001 C CNN
 	1    4950 2150
@@
 $EndComp
 $Comp
-L Device:R R?
+L Device:R R20
 U 1 1 5F5C5A5C
 P 4950 2650
-F 0 "R?" V 4743 2650 50  0000 C CNN
-F 1 "1K" V 4834 2650 50  0000 C CNN
-F 2 "" V 4880 2650 50  0001 C CNN
+F 0 "R20" V 4743 2650 50  0000 C CNN
+F 1 "1k" V 4834 2650 50  0000 C CNN
+F 2 "Resistor_SMD:R_0402_1005Metric" V 4880 2650 50  0001 C CNN
 F 3 "~" H 4950 2650 50  0001 C CNN
 	1    4950 2650
@@
 $EndComp
 $Comp
-L Device:CP C?
+L Device:CP C57
 U 1 1 5F5C5F2C
 P 7400 2150
-F 0 "C?" V 7145 2150 50  0000 C CNN
-F 1 "10.0" V 7236 2150 50  0000 C CNN
+F 0 "C57" V 7145 2150 50  0000 C CNN
+F 1 "10.0uF" V 7236 2150 50  0000 C CNN
 F 2 "" H 7438 2000 50  0001 C CNN
 F 3 "~" H 7400 2150 50  0001 C CNN
@@
 $EndComp
 $Comp
-L Device:CP C?
+L Device:CP C58
 U 1 1 5F5C6BAA
 P 7400 2650
-F 0 "C?" V 7145 2650 50  0000 C CNN
-F 1 "10.0" V 7236 2650 50  0000 C CNN
+F 0 "C58" V 7145 2650 50  0000 C CNN
+F 1 "10.0uF" V 7236 2650 50  0000 C CNN
 F 2 "" H 7438 2500 50  0001 C CNN
 F 3 "~" H 7400 2650 50  0001 C CNN
@@
 	6850 2150 5850 2150
 $Comp
-L power:GND #PWR?
+L power:GND #PWR036
 U 1 1 5F5CDE29
 P 6900 3150
-F 0 "#PWR?" H 6900 2900 50  0001 C CNN
+F 0 "#PWR036" H 6900 2900 50  0001 C CNN
 F 1 "GND" H 6905 2977 50  0000 C CNN
 F 2 "" H 6900 3150 50  0001 C CNN
@@
 $EndComp
 $Comp
-L power:GND #PWR?
+L power:GND #PWR034
 U 1 1 5F5CE47F
 P 6850 1600
-F 0 "#PWR?" H 6850 1350 50  0001 C CNN
+F 0 "#PWR034" H 6850 1350 50  0001 C CNN
 F 1 "GND" H 6855 1427 50  0000 C CNN
 F 2 "" H 6850 1600 50  0001 C CNN
@@
 Wire Wire Line
 	7550 2650 7900 2650
+$Comp
+L Device:R R22
+U 1 1 5F5C4893
+P 5850 2900
+F 0 "R22" H 5920 2946 50  0000 L CNN
+F 1 "2k" H 5920 2855 50  0000 L CNN
+F 2 "Resistor_SMD:R_0402_1005Metric" V 5780 2900 50  0001 C CNN
+F 3 "~" H 5850 2900 50  0001 C CNN
+	1    5850 2900
+	1    0    0    -1
+$EndComp
 $EndSCHEMATC

Commit message: updated BOM
Parts:
- removed C57, C58: 10.0uF, symbol Device:CP
- removed R16, R17: 4.7k, Resistor_SMD:R_0402_1005Metric, symbol Device:R
- removed R18, R23: 5.1k, Resistor_SMD:R_0402_1005Metric, symbol Device:R
- removed R19, R20: 1k, Resistor_SMD:R_0402_1005Metric, symbol Device:R
- removed R21, R22: 2k, Resistor_SMD:R_0402_1005Metric, symbol Device:R
- added C57, C58: 10uF, CAPC1005X55N, symbol SamacSys_Parts:10uF
- added R16, R23: 5.1k, RESC1005X40N, symbol SamacSys_Parts:5.1k
- added R17, R18: 4.7k, RESC1005X35N, symbol SamacSys_Parts:4.7k
- added R19, R20: 1k, RESC1005X35N, symbol SamacSys_Parts:1k
- added R21, R22: 2k, RESC1005X35N, symbol SamacSys_Parts:2k
Connections:
- net GND: now also R16.1, R23.2
- net SOUND: now also R17.1, R18.1
- net SOUND_LEFT: now also C58.1
- net SOUND_RIGHT: now also C57.1
- net at U2.3 (A): now also R19.2
- net at U2.38 (C): now also R20.2
- net at U2.4 (B): now also R21.2, R22.2
- new net: C57.2, R16.2, R18.2, R19.1, R22.1
- new net: C58.2, R17.2, R20.1, R21.1, R23.1
