File: zx/pentagon 128 portable/schematic/Pentagon128 portable/CPU.sch (KiCad schematic (older format))
At the start: 5 parts

Commit message: some reordering in the main project
Parts:
- removed IC?: GLS29EE010-70-4C-PHE, DIP1556W56P254L4191H508Q32N, symbol pentagon128_portable:GLS29EE010-70-4C-PHE
- removed R? (x2): 10K, symbol Device:R
- removed U?: Z80CPU, symbol CPU:Z80CPU
- removed U?: IS61C5128AS-25TLI, Package_SO:TSOP-II-32_21.0x10.2mm_P1.27mm, symbol Memory_RAM:IS61C5128AS-25TLI
- added C1, C10, C2, C3, C4, C5, C6, C7, C8, C9: 0.1uF, Capacitor_SMD:C_0402_1005Metric, symbol Device:C_Small
- added IC1: Z84C0020AEG, SamacSys_Parts:QFP80P1200X1200X160-44N, symbol SamacSys_Parts:Z84C0020AEG
- added IC2, IC3, IC4, IC5, IC6: TXB0108PWR, SamacSys_Parts:SOP65P640X120-20N, symbol SamacSys_Parts:TXB0108PWR
- added R1, R2: 10k, Resistor_SMD:R_0402_1005Metric, symbol Device:R_Small
- added R3, R4, R5, R6, R7: 50k, Resistor_SMD:R_0402_1005Metric, symbol Device:R_Small
Connections:
- net labels added: +3.3V, +5V_A0, +5V_A1, +5V_A10, +5V_A11, +5V_A12, +5V_A13, +5V_A14, +5V_A15, +5V_A2, +5V_A3, +5V_A4, +5V_A5, +5V_A6, +5V_A7, +5V_A8, +5V_A9, +5V_CLK, +5V_D0, +5V_D1, +5V_D2, +5V_D3, +5V_D4, +5V_D5, +5V_D6, +5V_D7, CLK, ~+5V_HALT, ~+5V_INT, ~+5V_IORQ, ~+5V_M1, ~+5V_MREQ, ~+5V_NMI, ~+5V_RD, ~+5V_RESET, ~+5V_RFSH, ~+5V_WR, ~HALT, ~RFSH
- net labels removed: RAM_PG0, RAM_PG1, RAM_PG2, RAM_PG3, RAM_PG4, ROM_PG0, ROM_PG1, ROM_PG2, ~CLK, ~RAM_CE, ~RAM_OE, ~RAM_WE, ~ROM_CE, ~ROM_OE, ~ROM_WE
- wire segments 103 -> 162
- no-connect marks 5 -> 4
Other:
- note added: "1.00"
- note added: "CPU"

Commit message: updated schemes
Parts:
- renumbered R3 to R1, R7 to R2, R1 to R3, R5 to R4, R2 to R5, R4 to R6, R6 to R7
Changed lines of the file:
@@
 ~+5V_NMI
 $Comp
-L Device:R_Small R1
+L Device:R_Small R3
 U 1 1 5F69C685
 P 5450 5150
-F 0 "R1" V 5254 5150 50  0000 C CNN
+F 0 "R3" V 5254 5150 50  0000 C CNN
 F 1 "10k" V 5345 5150 50  0000 C CNN
 F 2 "Resistor_SMD:R_0402_1005Metric" H 5450 5150 50  0001 C CNN
@@
 	5150 4600 5150 5150
 $Comp
-L Device:R_Small R2
+L Device:R_Small R5
 U 1 1 5F6A22F7
 P 5450 5450
-F 0 "R2" V 5254 5450 50  0000 C CNN
+F 0 "R5" V 5254 5450 50  0000 C CNN
 F 1 "10k" V 5345 5450 50  0000 C CNN
 F 2 "Resistor_SMD:R_0402_1005Metric" H 5450 5450 50  0001 C CNN
@@
 ~+5V_RFSH
 $Comp
-L power:+5V #PWR0104
+L power:+5V #PWR07
 U 1 1 5F6DEA7A
 P 5700 5000
-F 0 "#PWR0104" H 5700 4850 50  0001 C CNN
+F 0 "#PWR07" H 5700 4850 50  0001 C CNN
 F 1 "+5V" H 5715 5173 50  0000 C CNN
 F 2 "" H 5700 5000 50  0001 C CNN
@@
 Connection ~ 10200 1500
 $Comp
-L power:GND #PWR0105
+L power:GND #PWR02
 U 1 1 5F7D448A
 P 9850 1500
-F 0 "#PWR0105" H 9850 1250 50  0001 C CNN
+F 0 "#PWR02" H 9850 1250 50  0001 C CNN
 F 1 "GND" H 9855 1327 50  0000 C CNN
 F 2 "" H 9850 1500 50  0001 C CNN
@@
 $EndComp
 $Comp
-L power:+5V #PWR0106
+L power:+5V #PWR01
 U 1 1 5F7D5047
 P 9850 1300
-F 0 "#PWR0106" H 9850 1150 50  0001 C CNN
+F 0 "#PWR01" H 9850 1150 50  0001 C CNN
 F 1 "+5V" H 9865 1473 50  0000 C CNN
 F 2 "" H 9850 1300 50  0001 C CNN
@@
 Connection ~ 10150 2300
 $Comp
-L power:GND #PWR0107
+L power:GND #PWR04
 U 1 1 5F7D8E4D
 P 9800 2300
-F 0 "#PWR0107" H 9800 2050 50  0001 C CNN
+F 0 "#PWR04" H 9800 2050 50  0001 C CNN
 F 1 "GND" H 9805 2127 50  0000 C CNN
 F 2 "" H 9800 2300 50  0001 C CNN
@@
 $EndComp
 $Comp
-L power:+3.3V #PWR0108
+L power:+3.3V #PWR03
 U 1 1 5F7F0A0A
 P 9800 2100
-F 0 "#PWR0108" H 9800 1950 50  0001 C CNN
+F 0 "#PWR03" H 9800 1950 50  0001 C CNN
 F 1 "+3.3V" H 9815 2273 50  0000 C CNN
 F 2 "" H 9800 2100 50  0001 C CNN
@@
 $EndComp
 $Comp
-L power:+3.3V #PWR0109
+L power:+3.3V #PWR05
 U 1 1 5F83733F
 P 800 3800
-F 0 "#PWR0109" H 800 3650 50  0001 C CNN
+F 0 "#PWR05" H 800 3650 50  0001 C CNN
 F 1 "+3.3V" H 815 3973 50  0000 C CNN
 F 2 "" H 800 3800 50  0001 C CNN
@@
 $EndComp
 $Comp
-L Device:R_Small R3
+L Device:R_Small R1
 U 1 1 5F837EEE
 P 900 3800
-F 0 "R3" H 841 3754 50  0000 R CNN
+F 0 "R1" H 841 3754 50  0000 R CNN
 F 1 "50k" H 841 3845 50  0000 R CNN
 F 2 "Resistor_SMD:R_0402_1005Metric" H 900 3800 50  0001 C CNN
@@
 $EndComp
 $Comp
-L power:+3.3V #PWR0114
+L power:+3.3V #PWR08
 U 1 1 5FD7662A
 P 6600 5300
-F 0 "#PWR0114" H 6600 5150 50  0001 C CNN
+F 0 "#PWR08" H 6600 5150 50  0001 C CNN
 F 1 "+3.3V" H 6615 5473 50  0000 C CNN
 F 2 "" H 6600 5300 50  0001 C CNN
@@
 $EndComp
 $Comp
-L Device:R_Small R5
+L Device:R_Small R4
 U 1 1 5FD76634
 P 6700 5300
-F 0 "R5" H 6641 5254 50  0000 R CNN
+F 0 "R4" H 6641 5254 50  0000 R CNN
 F 1 "50k" H 6641 5345 50  0000 R CNN
 F 2 "Resistor_SMD:R_0402_1005Metric" H 6700 5300 50  0001 C CNN
@@
 $EndComp
 $Comp
-L power:+3.3V #PWR0115
+L power:+3.3V #PWR09
 U 1 1 5FD8AD76
 P 800 5550
-F 0 "#PWR0115" H 800 5400 50  0001 C CNN
+F 0 "#PWR09" H 800 5400 50  0001 C CNN
 F 1 "+3.3V" H 815 5723 50  0000 C CNN
 F 2 "" H 800 5550 50  0001 C CNN
@@
 $EndComp
 $Comp
-L Device:R_Small R4
+L Device:R_Small R6
 U 1 1 5FD8AD80
 P 900 5550
-F 0 "R4" H 841 5504 50  0000 R CNN
+F 0 "R6" H 841 5504 50  0000 R CNN
 F 1 "50k" H 841 5595 50  0000 R CNN
 F 2 "Resistor_SMD:R_0402_1005Metric" H 900 5550 50  0001 C CNN
@@
 $EndComp
 $Comp
-L power:+3.3V #PWR0116
+L power:+3.3V #PWR010
 U 1 1 5FD9F753
 P 2600 6950
-F 0 "#PWR0116" H 2600 6800 50  0001 C CNN
+F 0 "#PWR010" H 2600 6800 50  0001 C CNN
 F 1 "+3.3V" H 2615 7123 50  0000 C CNN
 F 2 "" H 2600 6950 50  0001 C CNN
@@
 $EndComp
 $Comp
-L Device:R_Small R6
+L Device:R_Small R7
 U 1 1 5FD9F75D
 P 2700 6950
-F 0 "R6" H 2641 6904 50  0000 R CNN
+F 0 "R7" H 2641 6904 50  0000 R CNN
 F 1 "50k" H 2641 6995 50  0000 R CNN
 F 2 "Resistor_SMD:R_0402_1005Metric" H 2700 6950 50  0001 C CNN
@@
 $EndComp
 $Comp
-L power:+3.3V #PWR0117
+L power:+3.3V #PWR06
 U 1 1 5FDB5282
 P 6600 3900
-F 0 "#PWR0117" H 6600 3750 50  0001 C CNN
+F 0 "#PWR06" H 6600 3750 50  0001 C CNN
 F 1 "+3.3V" H 6615 4073 50  0000 C CNN
 F 2 "" H 6600 3900 50  0001 C CNN
@@
 $EndComp
 $Comp
-L Device:R_Small R7
+L Device:R_Small R2
 U 1 1 5FDB528C
 P 6700 3900
-F 0 "R7" H 6641 3854 50  0000 R CNN
+F 0 "R2" H 6641 3854 50  0000 R CNN
 F 1 "50k" H 6641 3945 50  0000 R CNN
 F 2 "Resistor_SMD:R_0402_1005Metric" H 6700 3900 50  0001 C CNN

Commit message: updated BOM
Parts:
- removed C1, C10, C2, C3, C4, C5, C6, C7, C8, C9: 0.1uF, Capacitor_SMD:C_0402_1005Metric, symbol Device:C_Small
- removed R1, R2, R4, R6, R7: 50k, Resistor_SMD:R_0402_1005Metric, symbol Device:R_Small
- removed R3, R5: 10k, Resistor_SMD:R_0402_1005Metric, symbol Device:R_Small
- added C1, C10, C2, C3, C4, C5, C6, C7, C8, C9: 100nF, CAPC1005X55N, symbol SamacSys_Parts:100nF
- added R1, R2, R4, R6, R7: 49.9k, RESC1005X37N, symbol SamacSys_Parts:49.9k
- added R3, R5: 10k, RESC1005X37N, symbol SamacSys_Parts:10k
