File: zx/pentagon 128 portable/schematic/Pentagon128 portable/kempston.sch (KiCad schematic (older format))
At the start: 11 parts

Commit message: updated schemes
Parts:
- removed U?: 74HC240, symbol 74xx:74HC240
- added IC15: 74HC240PW,118, SamacSys_Parts:SOP65P640X110-20N, symbol SamacSys_Parts:74HC240PW,118
- added J9: Conn_01x06, symbol Connector_Generic:Conn_01x06
- R24, R25, R26, R27, R28: renamed from R?; value 1K -> 1k; footprint (none) -> Resistor_SMD:R_0402_1005Metric
- gave numbers to parts that had none: 5
Connections:
- net labels added: DOWN, FIRE, LEFT, RIGHT, UP
- wire segments 60 -> 59
Other:
- moved on the sheet: R24, R25, R26, R27, R28

Commit message: updated BOM
Parts:
- removed R24, R25, R26, R27, R28: 1k, Resistor_SMD:R_0402_1005Metric, symbol Device:R
- added R24, R25, R26, R27, R28: 1k, RESC1005X35N, symbol SamacSys_Parts:1k
- renumbered IC15 to IC8, J9 to J4
Changed lines of the file:
@@
 	2050 4350 1800 4350
-$Comp
-L Device:R R26
-U 1 1 5F5D9DAE
-P 3900 2250
-F 0 "R26" H 3970 2296 50  0000 L CNN
-F 1 "1k" H 3970 2205 50  0000 L CNN
-F 2 "Resistor_SMD:R_0402_1005Metric" V 3830 2250 50  0001 C CNN
-F 3 "~" H 3900 2250 50  0001 C CNN
-	1    3900 2250
-	1    0    0    -1
-$EndComp
-$Comp
-L Device:R R27
-U 1 1 5F5DA57C
-P 4150 2250
-F 0 "R27" H 4220 2296 50  0000 L CNN
-F 1 "1k" H 4220 2205 50  0000 L CNN
-F 2 "Resistor_SMD:R_0402_1005Metric" V 4080 2250 50  0001 C CNN
-F 3 "~" H 4150 2250 50  0001 C CNN
-	1    4150 2250
-	1    0    0    -1
-$EndComp
-$Comp
-L Device:R R28
-U 1 1 5F5DA88E
-P 4400 2250
-F 0 "R28" H 4470 2296 50  0000 L CNN
-F 1 "1k" H 4470 2205 50  0000 L CNN
-F 2 "Resistor_SMD:R_0402_1005Metric" V 4330 2250 50  0001 C CNN
-F 3 "~" H 4400 2250 50  0001 C CNN
-	1    4400 2250
-	1    0    0    -1
-$EndComp
-$Comp
-L Device:R R25
-U 1 1 5F5DABAB
-P 3650 2250
-F 0 "R25" H 3720 2296 50  0000 L CNN
-F 1 "1k" H 3720 2205 50  0000 L CNN
-F 2 "Resistor_SMD:R_0402_1005Metric" V 3580 2250 50  0001 C CNN
-F 3 "~" H 3650 2250 50  0001 C CNN
-	1    3650 2250
-	1    0    0    -1
-$EndComp
-$Comp
-L Device:R R24
-U 1 1 5F5DB19C
-P 3400 2250
-F 0 "R24" H 3470 2296 50  0000 L CNN
-F 1 "1k" H 3470 2205 50  0000 L CNN
-F 2 "Resistor_SMD:R_0402_1005Metric" V 3330 2250 50  0001 C CNN
-F 3 "~" H 3400 2250 50  0001 C CNN
-	1    3400 2250
-	1    0    0    -1
-$EndComp
 $Comp
 L Switch:SW_Push SW3
@@
 	1800 4850 1800 5100
 $Comp
-L power:GND #PWR042
+L power:GND #PWR046
 U 1 1 5F5E8FDE
 P 1800 5650
-F 0 "#PWR042" H 1800 5400 50  0001 C CNN
+F 0 "#PWR046" H 1800 5400 50  0001 C CNN
 F 1 "GND" H 1805 5477 50  0000 C CNN
 F 2 "" H 1800 5650 50  0001 C CNN
@@
 Connection ~ 1800 5350
 $Comp
-L power:+5V #PWR043
+L power:+5V #PWR045
 U 1 1 5F5E9E08
-P 3900 2700
-F 0 "#PWR043" H 3900 2550 50  0001 C CNN
-F 1 "+5V" H 3915 2873 50  0000 C CNN
-F 2 "" H 3900 2700 50  0001 C CNN
-F 3 "" H 3900 2700 50  0001 C CNN
-	1    3900 2700
+P 3900 2600
+F 0 "#PWR045" H 3900 2450 50  0001 C CNN
+F 1 "+5V" H 3915 2773 50  0000 C CNN
+F 2 "" H 3900 2600 50  0001 C CNN
+F 3 "" H 3900 2600 50  0001 C CNN
+	1    3900 2600
 	-1   0    0    1
 $EndComp
 Wire Wire Line
-	3900 2400 3900 2550
-Wire Wire Line
-	3400 2400 3400 2550
-Wire Wire Line
-	3400 2550 3650 2550
-Connection ~ 3900 2550
-Wire Wire Line
-	3900 2550 3900 2700
-Wire Wire Line
-	3900 2550 4150 2550
-Wire Wire Line
-	4400 2550 4400 2400
-Wire Wire Line
-	4150 2400 4150 2550
-Connection ~ 4150 2550
-Wire Wire Line
-	4150 2550 4400 2550
-Wire Wire Line
-	3650 2400 3650 2550
-Connection ~ 3650 2550
-Wire Wire Line
-	3650 2550 3900 2550
+	3900 2300 3900 2450
+Wire Wire Line
+	3400 2300 3400 2450
+Wire Wire Line
+	3400 2450 3650 2450
+Connection ~ 3900 2450
+Wire Wire Line
+	3900 2450 3900 2600
+Wire Wire Line
+	3900 2450 4150 2450
+Wire Wire Line
+	4400 2450 4400 2300
+Wire Wire Line
+	4150 2300 4150 2450
+Connection ~ 4150 2450
+Wire Wire Line
+	4150 2450 4400 2450
+Wire Wire Line
+	3650 2300 3650 2450
+Connection ~ 3650 2450
+Wire Wire Line
+	3650 2450 3900 2450
 Text HLabel 6400 1250 0    50   Input ~ 0
 KEMPSTON_SELECT
@@
 D1
 $Comp
-L SamacSys_Parts:74HC240PW,118 IC15
+L SamacSys_Parts:74HC240PW,118 IC8
 U 1 1 5F74DE9C
 P 6800 1250
-F 0 "IC15" H 7350 1515 50  0000 C CNN
+F 0 "IC8" H 7350 1515 50  0000 C CNN
 F 1 "74HC240PW,118" H 7350 1424 50  0000 C CNN
 F 2 "SamacSys_Parts:SOP65P640X110-20N" H 7750 1350 50  0001 L CNN
@@
 Connection ~ 6400 1550
 $Comp
-L power:+5V #PWR0101
+L power:+5V #PWR042
 U 1 1 5F757A3D
 P 6400 1350
-F 0 "#PWR0101" H 6400 1200 50  0001 C CNN
+F 0 "#PWR042" H 6400 1200 50  0001 C CNN
 F 1 "+5V" V 6415 1523 50  0000 C CNN
 F 2 "" H 6400 1350 50  0001 C CNN
@@
 RIGHT
 $Comp
-L Connector_Generic:Conn_01x06 J9
+L Connector_Generic:Conn_01x06 J4
 U 1 1 5F7594DC
 P 5250 1750
-F 0 "J9" H 5330 1742 50  0000 L CNN
+F 0 "J4" H 5330 1742 50  0000 L CNN
 F 1 "Conn_01x06" H 5330 1651 50  0000 L CNN
 F 2 "" H 5250 1750 50  0001 C CNN
@@
 RIGHT
 $Comp
-L power:GND #PWR0102
+L power:GND #PWR043
 U 1 1 5F75EF52
 P 4800 2050
-F 0 "#PWR0102" H 4800 1800 50  0001 C CNN
+F 0 "#PWR043" H 4800 1800 50  0001 C CNN
 F 1 "GND" H 4805 1877 50  0000 C CNN
 F 2 "" H 4800 2050 50  0001 C CNN
@@
 	2450 5350 3100 5350
 $Comp
-L power:GND #PWR0103
+L power:GND #PWR044
 U 1 1 5F79EDA2
 P 6650 2350
-F 0 "#PWR0103" H 6650 2100 50  0001 C CNN
+F 0 "#PWR044" H 6650 2100 50  0001 C CNN
 F 1 "GND" H 6655 2177 50  0000 C CNN
 F 2 "" H 6650 2350 50  0001 C CNN
@@
 Wire Wire Line
 	6650 2150 6650 2350
+$Comp
+L SamacSys_Parts:1k R24
+U 1 1 5F941390
+P 3400 2200
+F 0 "R24" H 3459 2246 50  0000 L CNN
+F 1 "1k" H 3459 2155 50  0000 L CNN
+F 2 "RESC1005X35N" H 3450 2050 50  0001 L CNN
+F 3 "http://www.yageo.com/documents/recent/PYu-RT_1-to-0.01_RoHS_L_9.pdf" H 3450 1950 50  0001 L CNN
+F 4 "Thin Film Resistors - SMD 1K ohm 1% 1/16W" H 3450 1850 50  0001 L CNN "Description"
+F 5 "0.35" H 3450 1750 50  0001 L CNN "Height"
+F 6 "603-RT0402FRE071KL" H 3450 1650 50  0001 L CNN "Mouser Part Number"
+F 7 "https://www.mouser.co.uk/ProductDetail/Yageo/RT0402FRE071KL?qs=BXCcY9r%252B08AJmLKodK5LLA%3D%3D" H 3450 1550 50  0001 L CNN "Mouser Price/Stock"
+F 8 "YAGEO (PHYCOMP)" H 3450 1450 50  0001 L CNN "Manufacturer_Name"
+F 9 "RT0402FRE071KL" H 3450 1350 50  0001 L CNN "Manufacturer_Part_Number"
+	1    3400 2200
+	1    0    0    -1
+$EndComp
+$Comp
+L SamacSys_Parts:1k R25
+U 1 1 5F941FA0
+P 3650 2200
+F 0 "R25" H 3709 2246 50  0000 L CNN
+F 1 "1k" H 3709 2155 50  0000 L CNN
+F 2 "RESC1005X35N" H 3700 2050 50  0001 L CNN
+F 3 "http://www.yageo.com/documents/recent/PYu-RT_1-to-0.01_RoHS_L_9.pdf" H 3700 1950 50  0001 L CNN
+F 4 "Thin Film Resistors - SMD 1K ohm 1% 1/16W" H 3700 1850 50  0001 L CNN "Description"
+F 5 "0.35" H 3700 1750 50  0001 L CNN "Height"
+F 6 "603-RT0402FRE071KL" H 3700 1650 50  0001 L CNN "Mouser Part Number"
+F 7 "https://www.mouser.co.uk/ProductDetail/Yageo/RT0402FRE071KL?qs=BXCcY9r%252B08AJmLKodK5LLA%3D%3D" H 3700 1550 50  0001 L CNN "Mouser Price/Stock"
+F 8 "YAGEO (PHYCOMP)" H 3700 1450 50  0001 L CNN "Manufacturer_Name"
+F 9 "RT0402FRE071KL" H 3700 1350 50  0001 L CNN "Manufacturer_Part_Number"
+	1    3650 2200
+	1    0    0    -1
+$EndComp
+$Comp
+L SamacSys_Parts:1k R26
+U 1 1 5F942199
+P 3900 2200
+F 0 "R26" H 3959 2246 50  0000 L CNN
+F 1 "1k" H 3959 2155 50  0000 L CNN
+F 2 "RESC1005X35N" H 3950 2050 50  0001 L CNN
+F 3 "http://www.yageo.com/documents/recent/PYu-RT_1-to-0.01_RoHS_L_9.pdf" H 3950 1950 50  0001 L CNN
+F 4 "Thin Film Resistors - SMD 1K ohm 1% 1/16W" H 3950 1850 50  0001 L CNN "Description"
+F 5 "0.35" H 3950 1750 50  0001 L CNN "Height"
+F 6 "603-RT0402FRE071KL" H 3950 1650 50  0001 L CNN "Mouser Part Number"
+F 7 "https://www.mouser.co.uk/ProductDetail/Yageo/RT0402FRE071KL?qs=BXCcY9r%252B08AJmLKodK5LLA%3D%3D" H 3950 1550 50  0001 L CNN "Mouser Price/Stock"
+F 8 "YAGEO (PHYCOMP)" H 3950 1450 50  0001 L CNN "Manufacturer_Name"
+F 9 "RT0402FRE071KL" H 3950 1350 50  0001 L CNN "Manufacturer_Part_Number"
+	1    3900 2200
+	1    0    0    -1
+$EndComp
+$Comp
+L SamacSys_Parts:1k R27
+U 1 1 5F9423D3
+P 4150 2200
+F 0 "R27" H 4209 2246 50  0000 L CNN
+F 1 "1k" H 4209 2155 50  0000 L CNN
+F 2 "RESC1005X35N" H 4200 2050 50  0001 L CNN
+F 3 "http://www.yageo.com/documents/recent/PYu-RT_1-to-0.01_RoHS_L_9.pdf" H 4200 1950 50  0001 L CNN
+F 4 "Thin Film Resistors - SMD 1K ohm 1% 1/16W" H 4200 1850 50  0001 L CNN "Description"
+F 5 "0.35" H 4200 1750 50  0001 L CNN "Height"
+F 6 "603-RT0402FRE071KL" H 4200 1650 50  0001 L CNN "Mouser Part Number"
+F 7 "https://www.mouser.co.uk/ProductDetail/Yageo/RT0402FRE071KL?qs=BXCcY9r%252B08AJmLKodK5LLA%3D%3D" H 4200 1550 50  0001 L CNN "Mouser Price/Stock"
+F 8 "YAGEO (PHYCOMP)" H 4200 1450 50  0001 L CNN "Manufacturer_Name"
+F 9 "RT0402FRE071KL" H 4200 1350 50  0001 L CNN "Manufacturer_Part_Number"
+	1    4150 2200
+	1    0    0    -1
+$EndComp
+$Comp
+L SamacSys_Parts:1k R28
+U 1 1 5F942862
+P 4400 2200
+F 0 "R28" H 4459 2246 50  0000 L CNN
+F 1 "1k" H 4459 2155 50  0000 L CNN
+F 2 "RESC1005X35N" H 4450 2050 50  0001 L CNN
+F 3 "http://www.yageo.com/documents/recent/PYu-RT_1-to-0.01_RoHS_L_9.pdf" H 4450 1950 50  0001 L CNN
+F 4 "Thin Film Resistors - SMD 1K ohm 1% 1/16W" H 4450 1850 50  0001 L CNN "Description"
+F 5 "0.35" H 4450 1750 50  0001 L CNN "Height"
+F 6 "603-RT0402FRE071KL" H 4450 1650 50  0001 L CNN "Mouser Part Number"
+F 7 "https://www.mouser.co.uk/ProductDetail/Yageo/RT0402FRE071KL?qs=BXCcY9r%252B08AJmLKodK5LLA%3D%3D" H 4450 1550 50  0001 L CNN "Mouser Price/Stock"
+F 8 "YAGEO (PHYCOMP)" H 4450 1450 50  0001 L CNN "Manufacturer_Name"
+F 9 "RT0402FRE071KL" H 4450 1350 50  0001 L CNN "Manufacturer_Part_Number"
+	1    4400 2200
+	1    0    0    -1
+$EndComp
 $EndSCHEMATC
