File: zx/pentagon 128 portable/schematic/Pentagon128 portable/memory.sch (KiCad schematic (older format))
At the start: 7 parts

Commit message: some reordering in the main project
Parts:
- removed IC?: SN74AHCT04D, SOIC127P600X175-14N, symbol SamacSys_Parts:SN74AHCT04D
- removed IC?: IS62C1024AL-35QLI, SOIC127P1412X305-32N, symbol SamacSys_Parts:IS62C1024AL-35QLI
- removed R? (x2): 10K, symbol Device:R
- removed U?: Z80CPU, symbol CPU:Z80CPU
Connections:
- net labels removed: A14, A15, ~CLK, ~INT, ~IORQ, ~M1, ~MREQ, ~NMI, ~RD, ~RESET, ~WR
- wire segments 102 -> 64
- no-connect marks 5 -> 2

Commit message: updated schemes
Parts:
- IC8: renamed from IC?; footprint DIP1556W56P254L4191H508Q32N -> Package_LCC:PLCC-32_11.4x14.0mm_P1.27mm
- IC9: renamed from IC?; footprint SOIC127P1176X120-32N -> SamacSys_Parts:SOIC127P1176X120-32N
Changed lines of the file:
@@
 $Descr A4 11693 8268
 encoding utf-8
-Sheet 7 14
+Sheet 10 14
 Title ""
 Date ""
@@
 	1100 7100 1200 7200
 $Comp
-L pentagon128_portable:GLS29EE010-70-4C-PHE IC?
+L pentagon128_portable:GLS29EE010-70-4C-PHE IC8
 U 1 1 5F4AAAD7
 P 8250 1350
-F 0 "IC?" H 8800 1615 50  0000 C CNN
+F 0 "IC8" H 8800 1615 50  0000 C CNN
 F 1 "GLS29EE010-70-4C-PHE" H 8800 1524 50  0000 C CNN
-F 2 "DIP1556W56P254L4191H508Q32N" H 9200 1450 50  0001 L CNN
+F 2 "Package_LCC:PLCC-32_11.4x14.0mm_P1.27mm" H 9200 1450 50  0001 L CNN
 F 3 "https://www.greenliant.com/dotAsset/40840.pdf" H 9200 1350 50  0001 L CNN
 F 4 "EEPROM 1MB, 5V, 70ns 128K x 8 Flash" H 9200 1250 50  0001 L CNN "Description"
@@
 ~RAM_WE
 $Comp
-L power:+5V #PWR?
+L power:+5V #PWR044
 U 1 1 5F5A1528
 P 9500 1200
-F 0 "#PWR?" H 9500 1050 50  0001 C CNN
+F 0 "#PWR044" H 9500 1050 50  0001 C CNN
 F 1 "+5V" H 9515 1373 50  0000 C CNN
 F 2 "" H 9500 1200 50  0001 C CNN
@@
 	9500 1350 9350 1350
 $Comp
-L power:GND #PWR?
+L power:GND #PWR046
 U 1 1 5F5A5F83
 P 8150 3050
-F 0 "#PWR?" H 8150 2800 50  0001 C CNN
+F 0 "#PWR046" H 8150 2800 50  0001 C CNN
 F 1 "GND" H 8155 2877 50  0000 C CNN
 F 2 "" H 8150 3050 50  0001 C CNN
@@
 	4650 2250 4650 2150
 $Comp
-L SamacSys_Parts:IS61C5128AS-25TLI IC?
+L SamacSys_Parts:IS61C5128AS-25TLI IC9
 U 1 1 5F88C91C
 P 3650 2250
-F 0 "IC?" H 4150 2515 50  0000 C CNN
+F 0 "IC9" H 4150 2515 50  0000 C CNN
 F 1 "IS61C5128AS-25TLI" H 4150 2424 50  0000 C CNN
-F 2 "SOIC127P1176X120-32N" H 4500 2350 50  0001 L CNN
+F 2 "SamacSys_Parts:SOIC127P1176X120-32N" H 4500 2350 50  0001 L CNN
 F 3 "https://componentsearchengine.com/Datasheets/1/IS61C5128AS-25TLI.pdf" H 4500 2250 50  0001 L CNN
 F 4 "SRAM 4M (512Kx8) 25ns Async SRAM" H 4500 2150 50  0001 L CNN "Description"
@@
 $EndComp
 $Comp
-L power:+5V #PWR?
+L power:+5V #PWR045
 U 1 1 5F5B424F
 P 4650 2150
-F 0 "#PWR?" H 4650 2000 50  0001 C CNN
+F 0 "#PWR045" H 4650 2000 50  0001 C CNN
 F 1 "+5V" H 4665 2323 50  0000 C CNN
 F 2 "" H 4650 2150 50  0001 C CNN
@@
 $EndComp
 $Comp
-L power:GND #PWR?
+L power:GND #PWR047
 U 1 1 5F5AAD46
 P 3650 3900
-F 0 "#PWR?" H 3650 3650 50  0001 C CNN
+F 0 "#PWR047" H 3650 3650 50  0001 C CNN
 F 1 "GND" H 3655 3727 50  0000 C CNN
 F 2 "" H 3650 3900 50  0001 C CNN

Commit message: updated BOM
Parts:
- renumbered IC9 to IC10, IC8 to IC9
Changed lines of the file:
@@
 	1100 7100 1200 7200
 $Comp
-L pentagon128_portable:GLS29EE010-70-4C-PHE IC8
+L pentagon128_portable:GLS29EE010-70-4C-PHE IC9
 U 1 1 5F4AAAD7
 P 8250 1350
-F 0 "IC8" H 8800 1615 50  0000 C CNN
+F 0 "IC9" H 8800 1615 50  0000 C CNN
 F 1 "GLS29EE010-70-4C-PHE" H 8800 1524 50  0000 C CNN
 F 2 "Package_LCC:PLCC-32_11.4x14.0mm_P1.27mm" H 9200 1450 50  0001 L CNN
@@
 ~RAM_WE
 $Comp
-L power:+5V #PWR044
+L power:+5V #PWR047
 U 1 1 5F5A1528
 P 9500 1200
-F 0 "#PWR044" H 9500 1050 50  0001 C CNN
+F 0 "#PWR047" H 9500 1050 50  0001 C CNN
 F 1 "+5V" H 9515 1373 50  0000 C CNN
 F 2 "" H 9500 1200 50  0001 C CNN
@@
 	9500 1350 9350 1350
 $Comp
-L power:GND #PWR046
+L power:GND #PWR049
 U 1 1 5F5A5F83
 P 8150 3050
-F 0 "#PWR046" H 8150 2800 50  0001 C CNN
+F 0 "#PWR049" H 8150 2800 50  0001 C CNN
 F 1 "GND" H 8155 2877 50  0000 C CNN
 F 2 "" H 8150 3050 50  0001 C CNN
@@
 	4650 2250 4650 2150
 $Comp
-L SamacSys_Parts:IS61C5128AS-25TLI IC9
+L SamacSys_Parts:IS61C5128AS-25TLI IC10
 U 1 1 5F88C91C
 P 3650 2250
-F 0 "IC9" H 4150 2515 50  0000 C CNN
+F 0 "IC10" H 4150 2515 50  0000 C CNN
 F 1 "IS61C5128AS-25TLI" H 4150 2424 50  0000 C CNN
 F 2 "SamacSys_Parts:SOIC127P1176X120-32N" H 4500 2350 50  0001 L CNN
@@
 $EndComp
 $Comp
-L power:+5V #PWR045
+L power:+5V #PWR048
 U 1 1 5F5B424F
 P 4650 2150
-F 0 "#PWR045" H 4650 2000 50  0001 C CNN
+F 0 "#PWR048" H 4650 2000 50  0001 C CNN
 F 1 "+5V" H 4665 2323 50  0000 C CNN
 F 2 "" H 4650 2150 50  0001 C CNN
@@
 $EndComp
 $Comp
-L power:GND #PWR047
+L power:GND #PWR050
 U 1 1 5F5AAD46
 P 3650 3900
-F 0 "#PWR047" H 3650 3650 50  0001 C CNN
+F 0 "#PWR050" H 3650 3650 50  0001 C CNN
 F 1 "GND" H 3655 3727 50  0000 C CNN
 F 2 "" H 3650 3900 50  0001 C CNN
