File: zx/pentagon 128 portable/schematic/Pentagon128 portable/peripheral.sch (KiCad schematic (older format))
At the start: 2 parts

Commit message: updated schemes
Parts:
- gave numbers to parts that had none: 2
Changed lines of the file:
@@
 $Descr A4 11693 8268
 encoding utf-8
-Sheet 12 14
+Sheet 14 14
 Title ""
 Date ""
@@
 P 1900 2000
 AR Path="/5F4A5D43/5F783155" Ref="J?"  Part="1"
-AR Path="/5F748573/5F783155" Ref="J?"  Part="1"
-F 0 "J?" H 1950 3017 50  0000 C CNN
+AR Path="/5F748573/5F783155" Ref="J7"  Part="1"
+F 0 "J7" H 1950 3017 50  0000 C CNN
 F 1 "Conn_02x17_Odd_Even" H 1950 2926 50  0000 C CNN
 F 2 "Connector_PinSocket_2.54mm:PinSocket_2x17_P2.54mm_Vertical" H 1900 2000 50  0001 C CNN
@@
 SDIO_CK
 $Comp
-L SamacSys_Parts:104031-0811 J?
+L SamacSys_Parts:104031-0811 J8
 U 1 1 5F7BADBD
 P 1500 3850
-F 0 "J?" H 2150 4115 50  0000 C CNN
+F 0 "J8" H 2150 4115 50  0000 C CNN
 F 1 "104031-0811" H 2150 4024 50  0000 C CNN
 F 2 "SamacSys_Parts:1040310811" H 2650 3950 50  0001 L CNN

Commit message: updated BOM
Parts:
- renumbered J7 to J8, J8 to J9
Changed lines of the file:
@@
 P 1900 2000
 AR Path="/5F4A5D43/5F783155" Ref="J?"  Part="1"
-AR Path="/5F748573/5F783155" Ref="J7"  Part="1"
-F 0 "J7" H 1950 3017 50  0000 C CNN
+AR Path="/5F748573/5F783155" Ref="J8"  Part="1"
+F 0 "J8" H 1950 3017 50  0000 C CNN
 F 1 "Conn_02x17_Odd_Even" H 1950 2926 50  0000 C CNN
 F 2 "Connector_PinSocket_2.54mm:PinSocket_2x17_P2.54mm_Vertical" H 1900 2000 50  0001 C CNN
@@
 SDIO_CK
 $Comp
-L SamacSys_Parts:104031-0811 J8
+L SamacSys_Parts:104031-0811 J9
 U 1 1 5F7BADBD
 P 1500 3850
-F 0 "J8" H 2150 4115 50  0000 C CNN
+F 0 "J9" H 2150 4115 50  0000 C CNN
 F 1 "104031-0811" H 2150 4024 50  0000 C CNN
 F 2 "SamacSys_Parts:1040310811" H 2650 3950 50  0001 L CNN
