File: zx/pentagon 128 portable/schematic/Pentagon128 portable/port_fe.sch (KiCad schematic (older format))
At the start: 25 parts

Commit message: some reordering in the main project
Parts:
- removed R? (x5): 10K, symbol Device:R
Connections:
- net KD0: no longer names the net of U?.17 (I3b)
- net KD1: no longer names the net of U?.15 (I2b)
- net KD2: no longer names the net of U?.13 (I1b)
- net KD3: no longer names the net of U?.11 (I0b)
- net KD4: no longer names the net of U?.8 (I3a)
Changed lines of the file:
@@
 $Descr A4 11693 8268
 encoding utf-8
-Sheet 6 8
+Sheet 9 14
 Title ""
 Date ""
@@
 Text Label 6800 1950 0    50   ~ 0
 TAPE_IN_DIGIT
-$Comp
-L Device:R R?
-U 1 1 5F5FDC64
-P 6650 2850
-F 0 "R?" H 6720 2896 50  0000 L CNN
-F 1 "10K" H 6720 2805 50  0000 L CNN
-F 2 "" V 6580 2850 50  0001 C CNN
-F 3 "~" H 6650 2850 50  0001 C CNN
-	1    6650 2850
-	1    0    0    -1
-$EndComp
-$Comp
-L Device:R R?
-U 1 1 5F5FDD3D
-P 6400 2850
-F 0 "R?" H 6470 2896 50  0000 L CNN
-F 1 "10K" H 6470 2805 50  0000 L CNN
-F 2 "" V 6330 2850 50  0001 C CNN
-F 3 "~" H 6400 2850 50  0001 C CNN
-	1    6400 2850
-	1    0    0    -1
-$EndComp
-$Comp
-L Device:R R?
-U 1 1 5F5FE243
-P 6150 2850
-F 0 "R?" H 6220 2896 50  0000 L CNN
-F 1 "10K" H 6220 2805 50  0000 L CNN
-F 2 "" V 6080 2850 50  0001 C CNN
-F 3 "~" H 6150 2850 50  0001 C CNN
-	1    6150 2850
-	1    0    0    -1
-$EndComp
-$Comp
-L Device:R R?
-U 1 1 5F5FE4EC
-P 5900 2850
-F 0 "R?" H 5970 2896 50  0000 L CNN
-F 1 "10K" H 5970 2805 50  0000 L CNN
-F 2 "" V 5830 2850 50  0001 C CNN
-F 3 "~" H 5900 2850 50  0001 C CNN
-	1    5900 2850
-	1    0    0    -1
-$EndComp
-$Comp
-L Device:R R?
-U 1 1 5F5FE776
-P 5650 2850
-F 0 "R?" H 5720 2896 50  0000 L CNN
-F 1 "10K" H 5720 2805 50  0000 L CNN
-F 2 "" V 5580 2850 50  0001 C CNN
-F 3 "~" H 5650 2850 50  0001 C CNN
-	1    5650 2850
-	1    0    0    -1
-$EndComp
 Text HLabel 7000 3100 3    50   Input ~ 0
 FE_RD_ENABLE
@@
 	7000 2850 7000 2750
 Wire Wire Line
-	7300 2550 6650 2550
-Wire Wire Line
-	7300 2450 6400 2450
-Wire Wire Line
-	7300 2350 6150 2350
-Wire Wire Line
-	7300 2250 5900 2250
-$Comp
-L power:+5V #PWR?
-U 1 1 5F6067EE
-P 6150 3150
-F 0 "#PWR?" H 6150 3000 50  0001 C CNN
-F 1 "+5V" H 6165 3323 50  0000 C CNN
-F 2 "" H 6150 3150 50  0001 C CNN
-F 3 "" H 6150 3150 50  0001 C CNN
-	1    6150 3150
-	-1   0    0    1
-$EndComp
-Wire Wire Line
-	6150 3000 6150 3100
-Wire Wire Line
-	6650 3000 6650 3100
-Wire Wire Line
-	6650 3100 6400 3100
-Connection ~ 6150 3100
-Wire Wire Line
-	6150 3100 6150 3150
-Wire Wire Line
-	6400 3000 6400 3100
-Connection ~ 6400 3100
-Wire Wire Line
-	6400 3100 6150 3100
-Wire Wire Line
-	5650 3000 5650 3100
-Wire Wire Line
-	5650 3100 5900 3100
-Wire Wire Line
-	5900 3000 5900 3100
-Connection ~ 5900 3100
-Wire Wire Line
-	5900 3100 6150 3100
-Wire Wire Line
-	6650 2700 6650 2550
-Wire Wire Line
-	6400 2700 6400 2450
-Wire Wire Line
-	6150 2700 6150 2350
-Wire Wire Line
-	5900 2700 5900 2250
-Wire Wire Line
-	5650 2700 5650 2150
-Wire Wire Line
-	5650 2150 7300 2150
-Wire Wire Line
-	6650 2550 5350 2550
-Connection ~ 6650 2550
-Wire Wire Line
-	6400 2450 5350 2450
-Connection ~ 6400 2450
-Wire Wire Line
-	6150 2350 5350 2350
-Connection ~ 6150 2350
-Wire Wire Line
-	5900 2250 5350 2250
-Connection ~ 5900 2250
-Wire Wire Line
-	5650 2150 5350 2150
-Connection ~ 5650 2150
-Text HLabel 5350 2150 0    50   Input ~ 0
-KD4
-Text HLabel 5350 2250 0    50   Input ~ 0
-KD3
-Text HLabel 5350 2350 0    50   Input ~ 0
-KD2
-Text HLabel 5350 2450 0    50   Input ~ 0
-KD1
-Text HLabel 5350 2550 0    50   Input ~ 0
-KD0
-Wire Wire Line
 	8300 1850 8750 1850

Commit message: updated schemes
Parts:
- removed C? (x2): C, symbol Device:C
- removed D? (x4): D, symbol Device:D
- removed R?: R, symbol Device:R
- removed R?: 430, symbol Device:R
- removed U? (x3): 4049, symbol 4xxx:4049
- removed U?: 74LS74, symbol 74xx:74LS74
- added C70, C71: 0.1uF, symbol Device:C
- added D1, D2, D3, D4: 1N4148W-7-F, SamacSys_Parts:SOD3716X145N, symbol SamacSys_Parts:1N4148W-7-F
- added IC13: 74HCT3G14DP,125, SamacSys_Parts:SOP65P400X110-8N, symbol SamacSys_Parts:74HCT3G14DP,125
- added IC14: SN74LS74ANSRG4, SamacSys_Parts:SOIC127P780X200-14N, symbol SamacSys_Parts:SN74LS74ANSRG4
- added R34: 100k, Resistor_SMD:R_0402_1005Metric, symbol Device:R
- added R36: 430, Resistor_SMD:R_0402_1005Metric, symbol Device:R
- C68: renamed from C?; value CP -> 10.0
- C69: renamed from C?; value C -> 1.0
- C72: renamed from C?; value 0.22 -> 0.22uF
- C73: renamed from C?; value 0.1 -> 0.1uF
- R35: renamed from R?; value R -> 620; footprint (none) -> Resistor_SMD:R_0402_1005Metric
- R37: renamed from R?; value 10K -> 10k; footprint (none) -> Resistor_SMD:R_0402_1005Metric
- U10: renamed from U?; footprint (none) -> Package_SO:SSOP-20_5.3x7.2mm_P0.65mm; Manufacturer_Part_Number (none) -> SN74LS244DBR; Mouser Part Number (none) -> 595-SN74LS244DBR
- U12: renamed from U?; footprint (none) -> Package_SO:SOIC-20W_7.5x12.8mm_P1.27mm; Mouser Part Number (none) -> 595-SN74LS175DR
Connections:
- net +5V: now also IC14.1 (1~CLR), IC14.14 (VCC), IC14.4 (1~PRE), R36.2
- net D4: now also IC14.2 (1D)
- net FE_WR_ENABLE: now also IC14.3 (1CLK)
- net GND: now also D1.1, D3.2, IC14.7 (GND)
- net SOUND: now also IC14.5 (1Q), R36.1
- net TAPE_IN_DIGIT: now also IC13.5
- net at R35.1: now also D2.1, D4.2, IC13.1
- net at C68.1: now also D1.2, D3.1
- new net: C71.2, D2.2, D4.1, IC13.7
- new net: C70.1, IC13.2, R34.2
- new net: C70.2, IC13.3
- new net: C71.1, IC13.6, R34.1
- no-connect marks 0 -> 7
Other:
- note removed: "4049-К561ЛН2"
- moved on the sheet: C68, C69, R35, U10

Commit message: updated BOM
Parts:
- removed C68: 10.0, symbol Device:CP
- removed C69: 1.0, symbol Device:C
- removed C70, C71, C73: 0.1uF, symbol Device:C
- removed C72: 0.22uF, symbol Device:C
- removed R34: 100k, Resistor_SMD:R_0402_1005Metric, symbol Device:R
- removed R35: 620, Resistor_SMD:R_0402_1005Metric, symbol Device:R
- removed R36: 430, Resistor_SMD:R_0402_1005Metric, symbol Device:R
- removed R37: 10k, Resistor_SMD:R_0402_1005Metric, symbol Device:R
- added C68: 10uF, CAPC1005X55N, symbol SamacSys_Parts:10uF
- added C69: 1uF, CAPC1005X33N, symbol SamacSys_Parts:1uF
- added C70, C71, C73: 100nF, CAPC1005X55N, symbol SamacSys_Parts:100nF
- added C72: 0.22uF, CAPC1005X56N, symbol SamacSys_Parts:0.22uF
- added R35: 620, RESC1005X35N, symbol SamacSys_Parts:620
- added R36: 100k, RESC1005X40N, symbol SamacSys_Parts:100k
- added R37: 430, RESC1005X35N, symbol SamacSys_Parts:430
- added R38: 10k, RESC1005X37N, symbol SamacSys_Parts:10k
- renumbered IC13 to IC14, IC14 to IC15, U10 to U6, U12 to U7
Connections:
- net +5V: now also R37.1
- net GND: now also C73.1
- net SOUND: now also R37.2
- net TAPE_IN: now also C69.2
- net TAPE_OUT: now also R38.1
- net at D1.2, D3.1: now also C68.1
- net at D2.1, D4.2, IC14.1: now also R35.1
- net at D2.2, D4.1, IC14.7: now also C71.2
- net at IC14.2: now also C70.1, R36.2
- net at IC14.3: now also C70.2
- net at IC14.6: now also C71.1, R36.1
- net at U7.15 (Q3): now also C72.1
- new net: C72.2, C73.2, R38.2
- new net: C68.2, C69.1, R35.2
