File: zx/pentagon 128 portable/schematic/Pentagon128 portable/power.sch (KiCad schematic (older format))
At the start: 15 parts

Commit message: updated schemes
Parts:
- gave numbers to parts that had none: 15
Changed lines of the file:
@@
 $Descr A4 11693 8268
 encoding utf-8
-Sheet 10 14
+Sheet 12 14
 Title ""
 Date ""
@@
 $EndDescr
 $Comp
-L Regulator_Linear:LD1117S50TR_SOT223 U?
+L Regulator_Linear:LD1117S50TR_SOT223 U4
 U 1 1 5F6C7ABF
 P 2650 1300
-F 0 "U?" H 2650 1542 50  0000 C CNN
+F 0 "U4" H 2650 1542 50  0000 C CNN
 F 1 "LD1117S50TR_SOT223" H 2650 1451 50  0000 C CNN
 F 2 "Package_TO_SOT_SMD:SOT-223-3_TabPin2" H 2650 1500 50  0001 C CNN
@@
 $EndComp
 $Comp
-L Regulator_Linear:LD1117S33TR_SOT223 U?
+L Regulator_Linear:LD1117S33TR_SOT223 U5
 U 1 1 5F6C7AC5
 P 4950 1300
-F 0 "U?" H 4950 1542 50  0000 C CNN
+F 0 "U5" H 4950 1542 50  0000 C CNN
 F 1 "LD1117S33TR_SOT223" H 4950 1451 50  0000 C CNN
 F 2 "Package_TO_SOT_SMD:SOT-223-3_TabPin2" H 4950 1500 50  0001 C CNN
@@
 $EndComp
 $Comp
-L Connector_Generic:Conn_01x02 J?
+L Connector_Generic:Conn_01x02 J5
 U 1 1 5F6C7ACB
 P 1550 1400
-F 0 "J?" H 1468 1075 50  0000 C CNN
+F 0 "J5" H 1468 1075 50  0000 C CNN
 F 1 "Conn_01x02" H 1468 1166 50  0000 C CNN
 F 2 "Connector_PinHeader_2.54mm:PinHeader_1x02_P2.54mm_Vertical" H 1550 1400 50  0001 C CNN
@@
 $EndComp
 $Comp
-L Device:C_Small C?
+L Device:C_Small C61
 U 1 1 5F6C7AD1
 P 3450 1400
-F 0 "C?" H 3542 1446 50  0000 L CNN
+F 0 "C61" H 3542 1446 50  0000 L CNN
 F 1 "100nF" H 3542 1355 50  0000 L CNN
 F 2 "Capacitor_SMD:C_0402_1005Metric" H 3450 1400 50  0001 C CNN
@@
 $EndComp
 $Comp
-L Device:CP_Small C?
+L Device:CP_Small C59
 U 1 1 5F6C7AD7
 P 2100 1400
-F 0 "C?" H 2188 1446 50  0000 L CNN
+F 0 "C59" H 2188 1446 50  0000 L CNN
 F 1 "10uF" H 2188 1355 50  0000 L CNN
 F 2 "Capacitor_SMD:C_0402_1005Metric" H 2100 1400 50  0001 C CNN
@@
 $EndComp
 $Comp
-L power:GND #PWR?
+L power:GND #PWR058
 U 1 1 5F6C7ADD
 P 2650 1750
-F 0 "#PWR?" H 2650 1500 50  0001 C CNN
+F 0 "#PWR058" H 2650 1500 50  0001 C CNN
 F 1 "GND" H 2655 1577 50  0000 C CNN
 F 2 "" H 2650 1750 50  0001 C CNN
@@
 Connection ~ 2100 1300
 $Comp
-L Device:CP_Small C?
+L Device:CP_Small C60
 U 1 1 5F6C7AED
 P 3100 1400
-F 0 "C?" H 3188 1446 50  0000 L CNN
+F 0 "C60" H 3188 1446 50  0000 L CNN
 F 1 "10uF" H 3188 1355 50  0000 L CNN
 F 2 "Capacitor_SMD:C_0402_1005Metric" H 3100 1400 50  0001 C CNN
@@
 +VIN
 $Comp
-L power:+5V #PWR?
+L power:+5V #PWR056
 U 1 1 5F6C7AFC
 P 3450 1300
-F 0 "#PWR?" H 3450 1150 50  0001 C CNN
+F 0 "#PWR056" H 3450 1150 50  0001 C CNN
 F 1 "+5V" H 3465 1473 50  0000 C CNN
 F 2 "" H 3450 1300 50  0001 C CNN
@@
 Connection ~ 3450 1300
 $Comp
-L Device:C_Small C?
+L Device:C_Small C64
 U 1 1 5F6C7B03
 P 5750 1400
-F 0 "C?" H 5842 1446 50  0000 L CNN
+F 0 "C64" H 5842 1446 50  0000 L CNN
 F 1 "100nF" H 5842 1355 50  0000 L CNN
 F 2 "Capacitor_SMD:C_0402_1005Metric" H 5750 1400 50  0001 C CNN
@@
 $EndComp
 $Comp
-L Device:CP_Small C?
+L Device:CP_Small C62
 U 1 1 5F6C7B09
 P 4400 1400
-F 0 "C?" H 4488 1446 50  0000 L CNN
+F 0 "C62" H 4488 1446 50  0000 L CNN
 F 1 "10uF" H 4488 1355 50  0000 L CNN
 F 2 "Capacitor_SMD:C_0402_1005Metric" H 4400 1400 50  0001 C CNN
@@
 $EndComp
 $Comp
-L power:GND #PWR?
+L power:GND #PWR059
 U 1 1 5F6C7B0F
 P 4950 1750
-F 0 "#PWR?" H 4950 1500 50  0001 C CNN
+F 0 "#PWR059" H 4950 1500 50  0001 C CNN
 F 1 "GND" H 4955 1577 50  0000 C CNN
 F 2 "" H 4950 1750 50  0001 C CNN
@@
 Connection ~ 4400 1300
 $Comp
-L Device:CP_Small C?
+L Device:CP_Small C63
 U 1 1 5F6C7B1B
 P 5400 1400
-F 0 "C?" H 5488 1446 50  0000 L CNN
+F 0 "C63" H 5488 1446 50  0000 L CNN
 F 1 "10uF" H 5488 1355 50  0000 L CNN
 F 2 "Capacitor_SMD:C_0402_1005Metric" H 5400 1400 50  0001 C CNN
@@
 	3450 1300 4400 1300
 $Comp
-L power:+3.3V #PWR?
+L power:+3.3V #PWR057
 U 1 1 5F6C7B2D
 P 5750 1300
-F 0 "#PWR?" H 5750 1150 50  0001 C CNN
+F 0 "#PWR057" H 5750 1150 50  0001 C CNN
 F 1 "+3.3V" H 5765 1473 50  0000 C CNN
 F 2 "" H 5750 1300 50  0001 C CNN
@@
 P 1750 2950
 AR Path="/5F4A5D43/5F825CE5" Ref="#PWR?"  Part="1"
-AR Path="/5F64EC48/5F825CE5" Ref="#PWR?"  Part="1"
-F 0 "#PWR?" H 1750 2800 50  0001 C CNN
+AR Path="/5F64EC48/5F825CE5" Ref="#PWR062"  Part="1"
+F 0 "#PWR062" H 1750 2800 50  0001 C CNN
 F 1 "+5V" H 1765 3123 50  0000 C CNN
 F 2 "" H 1750 2950 50  0001 C CNN
@@
 P 1900 3600
 AR Path="/5F4A5D43/5F825CEB" Ref="#PWR?"  Part="1"
-AR Path="/5F64EC48/5F825CEB" Ref="#PWR?"  Part="1"
-F 0 "#PWR?" H 1900 3350 50  0001 C CNN
+AR Path="/5F64EC48/5F825CEB" Ref="#PWR064"  Part="1"
+F 0 "#PWR064" H 1900 3350 50  0001 C CNN
 F 1 "GND" H 1905 3427 50  0000 C CNN
 F 2 "" H 1900 3600 50  0001 C CNN
@@
 P 1650 3300
 AR Path="/5F4A5D43/5F825CF1" Ref="R?"  Part="1"
-AR Path="/5F64EC48/5F825CF1" Ref="R?"  Part="1"
-F 0 "R?" H 1709 3346 50  0000 L CNN
+AR Path="/5F64EC48/5F825CF1" Ref="R33"  Part="1"
+F 0 "R33" H 1709 3346 50  0000 L CNN
 F 1 "100k" H 1709 3255 50  0000 L CNN
 F 2 "Resistor_SMD:R_0402_1005Metric" H 1650 3300 50  0001 C CNN
@@
 P 1900 3000
 AR Path="/5F4A5D43/5F825CFD" Ref="J?"  Part="1"
-AR Path="/5F64EC48/5F825CFD" Ref="J?"  Part="1"
-F 0 "J?" H 2350 3265 50  0000 C CNN
+AR Path="/5F64EC48/5F825CFD" Ref="J6"  Part="1"
+F 0 "J6" H 2350 3265 50  0000 C CNN
 F 1 "10033526-N3212LF" H 2350 3174 50  0000 C CNN
 F 2 "SamacSys_Parts:10033526N3212LF" H 2650 3100 50  0001 L CNN
@@
 	1450 3600 1900 3600
 $Comp
-L Regulator_Linear:LD1117S33TR_SOT223 U?
+L Regulator_Linear:LD1117S33TR_SOT223 U6
 U 1 1 5F88CF06
 P 4500 2900
-F 0 "U?" H 4500 3142 50  0000 C CNN
+F 0 "U6" H 4500 3142 50  0000 C CNN
 F 1 "LD1117S33TR_SOT223" H 4500 3051 50  0000 C CNN
 F 2 "Package_TO_SOT_SMD:SOT-223-3_TabPin2" H 4500 3100 50  0001 C CNN
@@
 $EndComp
 $Comp
-L Device:CP_Small C?
+L Device:CP_Small C65
 U 1 1 5F88CF0C
 P 3900 3050
-F 0 "C?" H 3988 3096 50  0000 L CNN
+F 0 "C65" H 3988 3096 50  0000 L CNN
 F 1 "10uF" H 3988 3005 50  0000 L CNN
 F 2 "Capacitor_SMD:C_0402_1005Metric" H 3900 3050 50  0001 C CNN
@@
 $EndComp
 $Comp
-L Device:CP_Small C?
+L Device:CP_Small C66
 U 1 1 5F88CF12
 P 4950 3050
-F 0 "C?" H 5038 3096 50  0000 L CNN
+F 0 "C66" H 5038 3096 50  0000 L CNN
 F 1 "10uF" H 5038 3005 50  0000 L CNN
 F 2 "Capacitor_SMD:C_0402_1005Metric" H 4950 3050 50  0001 C CNN
@@
 $EndComp
 $Comp
-L power:GND #PWR?
+L power:GND #PWR063
 U 1 1 5F88CF18
 P 4500 3350
-F 0 "#PWR?" H 4500 3100 50  0001 C CNN
+F 0 "#PWR063" H 4500 3100 50  0001 C CNN
 F 1 "GND" H 4505 3177 50  0000 C CNN
 F 2 "" H 4500 3350 50  0001 C CNN
@@
 $EndComp
 $Comp
-L Device:C_Small C?
+L Device:C_Small C67
 U 1 1 5F88CF1E
 P 5350 3050
-F 0 "C?" H 5442 3096 50  0000 L CNN
+F 0 "C67" H 5442 3096 50  0000 L CNN
 F 1 "100nF" H 5442 3005 50  0000 L CNN
 F 2 "Capacitor_SMD:C_0402_1005Metric" H 5350 3050 50  0001 C CNN
@@
 Connection ~ 3900 2900
 $Comp
-L power:+5V #PWR?
+L power:+5V #PWR060
 U 1 1 5F88CF39
 P 3750 2900
-F 0 "#PWR?" H 3750 2750 50  0001 C CNN
+F 0 "#PWR060" H 3750 2750 50  0001 C CNN
 F 1 "+5V" H 3765 3073 50  0000 C CNN
 F 2 "" H 3750 2900 50  0001 C CNN
@@
 VDD_MCU
 $Comp
-L power:+3.3V #PWR?
+L power:+3.3V #PWR061
 U 1 1 5F88CF40
 P 5850 2900
-F 0 "#PWR?" H 5850 2750 50  0001 C CNN
+F 0 "#PWR061" H 5850 2750 50  0001 C CNN
 F 1 "+3.3V" H 5865 3073 50  0000 C CNN
 F 2 "" H 5850 2900 50  0001 C CNN

Commit message: updated BOM
Parts:
- removed C59, C60, C62, C63, C65, C66: 10uF, Capacitor_SMD:C_0402_1005Metric, symbol Device:CP_Small
- removed C61, C64, C67: 100nF, Capacitor_SMD:C_0402_1005Metric, symbol Device:C_Small
- removed R33: 100k, Resistor_SMD:R_0402_1005Metric, symbol Device:R_Small
- removed U4: LD1117S50TR_SOT223, Package_TO_SOT_SMD:SOT-223-3_TabPin2, symbol Regulator_Linear:LD1117S50TR_SOT223
- removed U5, U6: LD1117S33TR_SOT223, Package_TO_SOT_SMD:SOT-223-3_TabPin2, symbol Regulator_Linear:LD1117S33TR_SOT223
- added C59, C60, C62, C63, C65, C66: 10uF, CAPC1005X55N, symbol SamacSys_Parts:10uF
- added C61, C64, C67: 100nF, CAPC1005X55N, symbol SamacSys_Parts:100nF
- added IC16: LD1117S50TR, SOT230P700X190-4N, symbol SamacSys_Parts:LD1117S50TR
- added IC17, IC18: LD1117S33TR, SOT230P700X190-4N, symbol SamacSys_Parts:LD1117S33TR
- added R34: 100k, RESC1005X40N, symbol SamacSys_Parts:100k
- renumbered J5 to J6, J6 to J7
Connections:
- wire segments 53 -> 55
