File: zx/pentagon 128 portable/schematic/Pentagon128 portable/stm32_cpu.sch (KiCad schematic (older format))
At the start: 12 parts

Commit message: updated schemes
Parts:
- gave numbers to parts that had none: 12
Changed lines of the file:
@@
 Comment4 ""
 $EndDescr
-$Comp
-L MCU_ST_STM32F4:STM32F469IITx U?
-U 1 1 5F9BCB38
-P 3450 5300
-AR Path="/5F4A5D43/5F9BCB38" Ref="U?"  Part="1"
-AR Path="/5F4A5D43/5F7467A7/5F9BCB38" Ref="U?"  Part="1"
-F 0 "U?" H 4600 900 50  0000 C CNN
-F 1 "STM32F469IITx" H 2400 900 50  0000 C CNN
-F 2 "Package_QFP:LQFP-176_24x24mm_P0.5mm" H 2050 1000 50  0001 R CNN
-F 3 "http://www.st.com/st-web-ui/static/active/en/resource/technical/document/datasheet/DM00219980.pdf" H 3450 5300 50  0001 C CNN
-	1    3450 5300
-	1    0    0    -1
-$EndComp
 Wire Wire Line
 	4950 6300 5350 6300
@@
 P 2950 10000
 AR Path="/5F4A5D43/5F9BCBA7" Ref="#PWR?"  Part="1"
-AR Path="/5F4A5D43/5F7467A7/5F9BCBA7" Ref="#PWR?"  Part="1"
-F 0 "#PWR?" H 2950 9750 50  0001 C CNN
+AR Path="/5F4A5D43/5F7467A7/5F9BCBA7" Ref="#PWR017"  Part="1"
+F 0 "#PWR017" H 2950 9750 50  0001 C CNN
 F 1 "GND" H 2955 9827 50  0000 C CNN
 F 2 "" H 2950 10000 50  0001 C CNN
@@
 P 1450 1600
 AR Path="/5F4A5D43/5F9BCBAE" Ref="#PWR?"  Part="1"
-AR Path="/5F4A5D43/5F7467A7/5F9BCBAE" Ref="#PWR?"  Part="1"
-F 0 "#PWR?" H 1450 1350 50  0001 C CNN
+AR Path="/5F4A5D43/5F7467A7/5F9BCBAE" Ref="#PWR014"  Part="1"
+F 0 "#PWR014" H 1450 1350 50  0001 C CNN
 F 1 "GND" V 1455 1472 50  0000 R CNN
 F 2 "" H 1450 1600 50  0001 C CNN
@@
 P 1550 1600
 AR Path="/5F4A5D43/5F9BCBF8" Ref="R?"  Part="1"
-AR Path="/5F4A5D43/5F7467A7/5F9BCBF8" Ref="R?"  Part="1"
-F 0 "R?" V 1354 1600 50  0000 C CNN
+AR Path="/5F4A5D43/5F7467A7/5F9BCBF8" Ref="R10"  Part="1"
+F 0 "R10" V 1354 1600 50  0000 C CNN
 F 1 "10k" V 1445 1600 50  0000 C CNN
 F 2 "Resistor_SMD:R_0402_1005Metric" H 1550 1600 50  0001 C CNN
@@
 P -1950 10200
 AR Path="/5F4A5D43/5F9BCBFE" Ref="C?"  Part="1"
-AR Path="/5F4A5D43/5F7467A7/5F9BCBFE" Ref="C?"  Part="1"
-F 0 "C?" H -1858 10246 50  0000 L CNN
+AR Path="/5F4A5D43/5F7467A7/5F9BCBFE" Ref="C13"  Part="1"
+F 0 "C13" H -1858 10246 50  0000 L CNN
 F 1 "100nF" H -1858 10155 50  0000 L CNN
 F 2 "Capacitor_SMD:C_0402_1005Metric" H -1950 10200 50  0001 C CNN
@@
 P -1950 9750
 AR Path="/5F4A5D43/5F9BCC04" Ref="R?"  Part="1"
-AR Path="/5F4A5D43/5F7467A7/5F9BCC04" Ref="R?"  Part="1"
-F 0 "R?" H -1891 9796 50  0000 L CNN
+AR Path="/5F4A5D43/5F7467A7/5F9BCC04" Ref="R11"  Part="1"
+F 0 "R11" H -1891 9796 50  0000 L CNN
 F 1 "100k" H -1891 9705 50  0000 L CNN
 F 2 "Resistor_SMD:R_0402_1005Metric" H -1950 9750 50  0001 C CNN
@@
 P -1400 10300
 AR Path="/5F4A5D43/5F9BCC0A" Ref="SW?"  Part="1"
-AR Path="/5F4A5D43/5F7467A7/5F9BCC0A" Ref="SW?"  Part="1"
-F 0 "SW?" V -1446 10448 50  0000 L CNN
+AR Path="/5F4A5D43/5F7467A7/5F9BCC0A" Ref="SW1"  Part="1"
+F 0 "SW1" V -1446 10448 50  0000 L CNN
 F 1 "SW_Push" V -1355 10448 50  0000 L CNN
 F 2 "Button_Switch_SMD:SW_DIP_SPSTx01_Slide_6.7x4.1mm_W6.73mm_P2.54mm_LowProfile_JPin" H -1400 10500 50  0001 C CNN
@@
 P -1950 9650
 AR Path="/5F4A5D43/5F9BCC14" Ref="#PWR?"  Part="1"
-AR Path="/5F4A5D43/5F7467A7/5F9BCC14" Ref="#PWR?"  Part="1"
-F 0 "#PWR?" H -1950 9500 50  0001 C CNN
+AR Path="/5F4A5D43/5F7467A7/5F9BCC14" Ref="#PWR016"  Part="1"
+F 0 "#PWR016" H -1950 9500 50  0001 C CNN
 F 1 "+3.3V" H -1935 9823 50  0000 C CNN
 F 2 "" H -1950 9650 50  0001 C CNN
@@
 P -1400 10750
 AR Path="/5F4A5D43/5F9BCC1C" Ref="#PWR?"  Part="1"
-AR Path="/5F4A5D43/5F7467A7/5F9BCC1C" Ref="#PWR?"  Part="1"
-F 0 "#PWR?" H -1400 10500 50  0001 C CNN
+AR Path="/5F4A5D43/5F7467A7/5F9BCC1C" Ref="#PWR018"  Part="1"
+F 0 "#PWR018" H -1400 10500 50  0001 C CNN
 F 1 "GND" H -1395 10577 50  0000 C CNN
 F 2 "" H -1400 10750 50  0001 C CNN
@@
 P 2300 850
 AR Path="/5F4A5D43/5F9BCC2A" Ref="J?"  Part="1"
-AR Path="/5F4A5D43/5F7467A7/5F9BCC2A" Ref="J?"  Part="1"
-F 0 "J?" H 2408 1039 50  0000 C CNN
+AR Path="/5F4A5D43/5F7467A7/5F9BCC2A" Ref="J1"  Part="1"
+F 0 "J1" H 2408 1039 50  0000 C CNN
 F 1 "Conn_01x03_Male" H 2408 1040 50  0001 C CNN
 F 2 "Connector_PinHeader_2.54mm:PinHeader_1x03_P2.54mm_Vertical" H 2300 850 50  0001 C CNN
@@
 P 750 1000
 AR Path="/5F4A5D43/5F9BCC34" Ref="#PWR?"  Part="1"
-AR Path="/5F4A5D43/5F7467A7/5F9BCC34" Ref="#PWR?"  Part="1"
-F 0 "#PWR?" H 750 750 50  0001 C CNN
+AR Path="/5F4A5D43/5F7467A7/5F9BCC34" Ref="#PWR012"  Part="1"
+F 0 "#PWR012" H 750 750 50  0001 C CNN
 F 1 "GND" V 755 872 50  0000 R CNN
 F 2 "" H 750 1000 50  0001 C CNN
@@
 P 2600 650
 AR Path="/5F4A5D43/5F9BCC3A" Ref="#PWR?"  Part="1"
-AR Path="/5F4A5D43/5F7467A7/5F9BCC3A" Ref="#PWR?"  Part="1"
-F 0 "#PWR?" H 2600 500 50  0001 C CNN
+AR Path="/5F4A5D43/5F7467A7/5F9BCC3A" Ref="#PWR011"  Part="1"
+F 0 "#PWR011" H 2600 500 50  0001 C CNN
 F 1 "+3.3V" H 2615 823 50  0000 C CNN
 F 2 "" H 2600 650 50  0001 C CNN
@@
 P 1100 1300
 AR Path="/5F4A5D43/5F9BCC42" Ref="R?"  Part="1"
-AR Path="/5F4A5D43/5F7467A7/5F9BCC42" Ref="R?"  Part="1"
-F 0 "R?" V 904 1300 50  0000 C CNN
+AR Path="/5F4A5D43/5F7467A7/5F9BCC42" Ref="R8"  Part="1"
+F 0 "R8" V 904 1300 50  0000 C CNN
 F 1 "10k" V 995 1300 50  0000 C CNN
 F 2 "Resistor_SMD:R_0402_1005Metric" H 1100 1300 50  0001 C CNN
@@
 P 950 1800
 AR Path="/5F4A5D43/5F9BCC4D" Ref="C?"  Part="1"
-AR Path="/5F4A5D43/5F7467A7/5F9BCC4D" Ref="C?"  Part="1"
-F 0 "C?" V 721 1800 50  0000 C CNN
+AR Path="/5F4A5D43/5F7467A7/5F9BCC4D" Ref="C11"  Part="1"
+F 0 "C11" V 721 1800 50  0000 C CNN
 F 1 "2.2uF" V 812 1800 50  0000 C CNN
 F 2 "Capacitor_SMD:C_1210_3225Metric_Pad1.42x2.65mm_HandSolder" H 950 1800 50  0001 C CNN
@@
 P 650 1900
 AR Path="/5F4A5D43/5F9BCC53" Ref="C?"  Part="1"
-AR Path="/5F4A5D43/5F7467A7/5F9BCC53" Ref="C?"  Part="1"
-F 0 "C?" V 421 1900 50  0000 C CNN
+AR Path="/5F4A5D43/5F7467A7/5F9BCC53" Ref="C12"  Part="1"
+F 0 "C12" V 421 1900 50  0000 C CNN
 F 1 "2.2uF" V 512 1900 50  0000 C CNN
 F 2 "Capacitor_SMD:C_1210_3225Metric_Pad1.42x2.65mm_HandSolder" H 650 1900 50  0001 C CNN
@@
 P 400 1900
 AR Path="/5F4A5D43/5F9BCC5E" Ref="#PWR?"  Part="1"
-AR Path="/5F4A5D43/5F7467A7/5F9BCC5E" Ref="#PWR?"  Part="1"
-F 0 "#PWR?" H 400 1650 50  0001 C CNN
+AR Path="/5F4A5D43/5F7467A7/5F9BCC5E" Ref="#PWR015"  Part="1"
+F 0 "#PWR015" H 400 1650 50  0001 C CNN
 F 1 "GND" V 405 1772 50  0000 R CNN
 F 2 "" H 400 1900 50  0001 C CNN
@@
 P 1300 2500
 AR Path="/5F4A5D43/5F9BCC74" Ref="J?"  Part="1"
-AR Path="/5F4A5D43/5F7467A7/5F9BCC74" Ref="J?"  Part="1"
-F 0 "J?" H 1408 2881 50  0000 C CNN
+AR Path="/5F4A5D43/5F7467A7/5F9BCC74" Ref="J2"  Part="1"
+F 0 "J2" H 1408 2881 50  0000 C CNN
 F 1 "DSI" H 1408 2790 50  0000 C CNN
 F 2 "Connector_PinHeader_2.54mm:PinHeader_1x06_P2.54mm_Vertical" H 1300 2500 50  0001 C CNN
@@
 P 1300 1400
 AR Path="/5F4A5D43/5F9BCCF6" Ref="R?"  Part="1"
-AR Path="/5F4A5D43/5F7467A7/5F9BCCF6" Ref="R?"  Part="1"
-F 0 "R?" V 1104 1400 50  0000 C CNN
+AR Path="/5F4A5D43/5F7467A7/5F9BCCF6" Ref="R9"  Part="1"
+F 0 "R9" V 1104 1400 50  0000 C CNN
 F 1 "10k" V 1195 1400 50  0000 C CNN
 F 2 "Resistor_SMD:R_0402_1005Metric" H 1300 1400 50  0001 C CNN
@@
 P 1200 1400
 AR Path="/5F4A5D43/5F9BCCFC" Ref="#PWR?"  Part="1"
-AR Path="/5F4A5D43/5F7467A7/5F9BCCFC" Ref="#PWR?"  Part="1"
-F 0 "#PWR?" H 1200 1250 50  0001 C CNN
+AR Path="/5F4A5D43/5F7467A7/5F9BCCFC" Ref="#PWR013"  Part="1"
+F 0 "#PWR013" H 1200 1250 50  0001 C CNN
 F 1 "+3.3V" V 1215 1528 50  0000 L CNN
 F 2 "" H 1200 1400 50  0001 C CNN
@@
 P 1100 350
 AR Path="/5F4A5D43/5F9BCD11" Ref="IC?"  Part="1"
-AR Path="/5F4A5D43/5F7467A7/5F9BCD11" Ref="IC?"  Part="1"
-F 0 "IC?" H 1944 396 50  0000 L CNN
+AR Path="/5F4A5D43/5F7467A7/5F9BCD11" Ref="IC7"  Part="1"
+F 0 "IC7" H 1944 396 50  0000 L CNN
 F 1 "1072" H 1944 305 50  0000 L CNN
 F 2 "SamacSys_Parts:1072" H 1750 750 50  0001 L CNN
@@
 Wire Wire Line
 	4050 9800 4150 9800
+$Comp
+L MCU_ST_STM32F4:STM32F469IITx U?
+U 1 1 5F9BCB38
+P 3450 5300
+AR Path="/5F4A5D43/5F9BCB38" Ref="U?"  Part="1"
+AR Path="/5F4A5D43/5F7467A7/5F9BCB38" Ref="U1"  Part="1"
+F 0 "U1" H 4600 900 50  0000 C CNN
+F 1 "STM32F469IITx" H 2400 900 50  0000 C CNN
+F 2 "Package_QFP:LQFP-176_24x24mm_P0.5mm" H 2050 1000 50  0001 R CNN
+F 3 "http://www.st.com/st-web-ui/static/active/en/resource/technical/document/datasheet/DM00219980.pdf" H 3450 5300 50  0001 C CNN
+	1    3450 5300
+	1    0    0    -1
+$EndComp
 $EndSCHEMATC

Commit message: updated BOM
Parts:
- removed C11, C12: 2.2uF, Capacitor_SMD:C_1210_3225Metric_Pad1.42x2.65mm_HandSolder, symbol Device:C_Small
- removed C13: 100nF, Capacitor_SMD:C_0402_1005Metric, symbol Device:C_Small
- removed R10, R8, R9: 10k, Resistor_SMD:R_0402_1005Metric, symbol Device:R_Small
- removed R11: 100k, Resistor_SMD:R_0402_1005Metric, symbol Device:R_Small
- added C11, C12: 2.2uF_tantalum, CAPPM3216X180N, symbol SamacSys_Parts:2.2uF_tantalum
- added C13: 100nF, CAPC1005X55N, symbol SamacSys_Parts:100nF
- added R10, R8, R9: 10k, RESC1005X37N, symbol SamacSys_Parts:10k
- added R11: 100k, RESC1005X40N, symbol SamacSys_Parts:100k
Changed lines of the file:
@@
 Wire Wire Line
 	1850 1200 1400 1200
-Wire Wire Line
-	1850 1400 1400 1400
 Text Label 1400 1200 0    50   ~ 0
 NRST
-$Comp
-L Device:R_Small R?
-U 1 1 5F9BCBF8
-P 1550 1600
-AR Path="/5F4A5D43/5F9BCBF8" Ref="R?"  Part="1"
-AR Path="/5F4A5D43/5F7467A7/5F9BCBF8" Ref="R10"  Part="1"
-F 0 "R10" V 1354 1600 50  0000 C CNN
-F 1 "10k" V 1445 1600 50  0000 C CNN
-F 2 "Resistor_SMD:R_0402_1005Metric" H 1550 1600 50  0001 C CNN
-F 3 "~" H 1550 1600 50  0001 C CNN
-	1    1550 1600
-	0    1    1    0
-$EndComp
-$Comp
-L Device:C_Small C?
-U 1 1 5F9BCBFE
-P -1950 10200
-AR Path="/5F4A5D43/5F9BCBFE" Ref="C?"  Part="1"
-AR Path="/5F4A5D43/5F7467A7/5F9BCBFE" Ref="C13"  Part="1"
-F 0 "C13" H -1858 10246 50  0000 L CNN
-F 1 "100nF" H -1858 10155 50  0000 L CNN
-F 2 "Capacitor_SMD:C_0402_1005Metric" H -1950 10200 50  0001 C CNN
-F 3 "~" H -1950 10200 50  0001 C CNN
-	1    -1950 10200
-	1    0    0    -1
-$EndComp
-$Comp
-L Device:R_Small R?
-U 1 1 5F9BCC04
-P -1950 9750
-AR Path="/5F4A5D43/5F9BCC04" Ref="R?"  Part="1"
-AR Path="/5F4A5D43/5F7467A7/5F9BCC04" Ref="R11"  Part="1"
-F 0 "R11" H -1891 9796 50  0000 L CNN
-F 1 "100k" H -1891 9705 50  0000 L CNN
-F 2 "Resistor_SMD:R_0402_1005Metric" H -1950 9750 50  0001 C CNN
-F 3 "~" H -1950 9750 50  0001 C CNN
-	1    -1950 9750
-	1    0    0    -1
-$EndComp
 $Comp
 L Switch:SW_Push SW?
@@
 Wire Wire Line
 	2600 750  2500 750
-$Comp
-L Device:R_Small R?
-U 1 1 5F9BCC42
-P 1100 1300
-AR Path="/5F4A5D43/5F9BCC42" Ref="R?"  Part="1"
-AR Path="/5F4A5D43/5F7467A7/5F9BCC42" Ref="R8"  Part="1"
-F 0 "R8" V 904 1300 50  0000 C CNN
-F 1 "10k" V 995 1300 50  0000 C CNN
-F 2 "Resistor_SMD:R_0402_1005Metric" H 1100 1300 50  0001 C CNN
-F 3 "~" H 1100 1300 50  0001 C CNN
-	1    1100 1300
-	0    1    1    0
-$EndComp
 Wire Wire Line
 	750  1000 850  1000
@@
 Wire Wire Line
 	1200 1300 1850 1300
-$Comp
-L Device:C_Small C?
-U 1 1 5F9BCC4D
-P 950 1800
-AR Path="/5F4A5D43/5F9BCC4D" Ref="C?"  Part="1"
-AR Path="/5F4A5D43/5F7467A7/5F9BCC4D" Ref="C11"  Part="1"
-F 0 "C11" V 721 1800 50  0000 C CNN
-F 1 "2.2uF" V 812 1800 50  0000 C CNN
-F 2 "Capacitor_SMD:C_1210_3225Metric_Pad1.42x2.65mm_HandSolder" H 950 1800 50  0001 C CNN
-F 3 "~" H 950 1800 50  0001 C CNN
-	1    950  1800
-	0    1    1    0
-$EndComp
-$Comp
-L Device:C_Small C?
-U 1 1 5F9BCC53
-P 650 1900
-AR Path="/5F4A5D43/5F9BCC53" Ref="C?"  Part="1"
-AR Path="/5F4A5D43/5F7467A7/5F9BCC53" Ref="C12"  Part="1"
-F 0 "C12" V 421 1900 50  0000 C CNN
-F 1 "2.2uF" V 512 1900 50  0000 C CNN
-F 2 "Capacitor_SMD:C_1210_3225Metric_Pad1.42x2.65mm_HandSolder" H 650 1900 50  0001 C CNN
-F 3 "~" H 650 1900 50  0001 C CNN
-	1    650  1900
-	0    1    1    0
-$EndComp
-Wire Wire Line
-	1850 1800 1050 1800
-Wire Wire Line
-	1850 1900 750  1900
-Wire Wire Line
-	850  1800 400  1800
 Wire Wire Line
 	400  1800 400  1900
@@
 PE15
 $Comp
-L Device:R_Small R?
-U 1 1 5F9BCCF6
-P 1300 1400
-AR Path="/5F4A5D43/5F9BCCF6" Ref="R?"  Part="1"
-AR Path="/5F4A5D43/5F7467A7/5F9BCCF6" Ref="R9"  Part="1"
-F 0 "R9" V 1104 1400 50  0000 C CNN
-F 1 "10k" V 1195 1400 50  0000 C CNN
-F 2 "Resistor_SMD:R_0402_1005Metric" H 1300 1400 50  0001 C CNN
-F 3 "~" H 1300 1400 50  0001 C CNN
-	1    1300 1400
-	0    1    1    0
-$EndComp
-$Comp
 L power:+3.3V #PWR?
 U 1 1 5F9BCCFC
@@
 	1    0    0    -1
 $EndComp
+$Comp
+L SamacSys_Parts:100nF C13
+U 1 1 5F796A70
+P -1950 10200
+F 0 "C13" H -1858 10246 50  0000 L CNN
+F 1 "100nF" H -1858 10155 50  0000 L CNN
+F 2 "CAPC1005X55N" H -1850 10050 50  0001 L CNN
+F 3 "https://content.kemet.com/datasheets/KEM_C1002_X7R_SMD.pdf" H -1850 9950 50  0001 L CNN
+F 4 "KEMET - C0402C104K9PACTU - CAP, MLCC, X5R, 0.1UF, 6.3V, 0402, REEL" H -1850 9850 50  0001 L CNN "Description"
+F 5 "0.55" H -1850 9750 50  0001 L CNN "Height"
+F 6 "80-C0402C104K9P" H -1850 9650 50  0001 L CNN "Mouser Part Number"
+F 7 "https://www.mouser.co.uk/ProductDetail/KEMET/C0402C104K9PACTU?qs=DBJr%252BvBUjU7yQ9iUbxvTPw%3D%3D" H -1850 9550 50  0001 L CNN "Mouser Price/Stock"
+F 8 "Kemet" H -1850 9450 50  0001 L CNN "Manufacturer_Name"
+F 9 "C0402C104K9PACTU" H -1850 9350 50  0001 L CNN "Manufacturer_Part_Number"
+	1    -1950 10200
+	1    0    0    -1
+$EndComp
+$Comp
+L SamacSys_Parts:2.2uF_tantalum C11
+U 1 1 5F842E04
+P 950 1800
+F 0 "C11" V 725 1800 50  0000 C CNN
+F 1 "2.2uF_tantalum" V 816 1800 50  0000 C CNN
+F 2 "CAPPM3216X180N" H 1050 1650 50  0001 L CNN
+F 3 "" H 1050 1550 50  0001 L CNN
+F 4 "Tantalum Capacitors - Solid SMD 10V 2.2uF 10% 1206 ESR=6.5Ohm AEC-Q200" H 1050 1450 50  0001 L CNN "Description"
+F 5 "1.8" H 1050 1350 50  0001 L CNN "Height"
+F 6 "581-TAJA225K010TNJ" H 1050 1250 50  0001 L CNN "Mouser Part Number"
+F 7 "https://www.mouser.co.uk/ProductDetail/AVX/TAJA225K010TNJ?qs=XLNwXgtzMM%2F9RK%2FJN7CZtw%3D%3D" H 1050 1150 50  0001 L CNN "Mouser Price/Stock"
+F 8 "AVX" H 1050 1050 50  0001 L CNN "Manufacturer_Name"
+F 9 "TAJA225K010TNJ" H 1050 950 50  0001 L CNN "Manufacturer_Part_Number"
+	1    950  1800
+	0    1    1    0
+$EndComp
+$Comp
+L SamacSys_Parts:2.2uF_tantalum C12
+U 1 1 5F843617
+P 650 1900
+F 0 "C12" V 750 1900 50  0000 C CNN
+F 1 "2.2uF_tantalum" V 850 2050 50  0000 C CNN
+F 2 "CAPPM3216X180N" H 750 1750 50  0001 L CNN
+F 3 "" H 750 1650 50  0001 L CNN
+F 4 "Tantalum Capacitors - Solid SMD 10V 2.2uF 10% 1206 ESR=6.5Ohm AEC-Q200" H 750 1550 50  0001 L CNN "Description"
+F 5 "1.8" H 750 1450 50  0001 L CNN "Height"
+F 6 "581-TAJA225K010TNJ" H 750 1350 50  0001 L CNN "Mouser Part Number"
+F 7 "https://www.mouser.co.uk/ProductDetail/AVX/TAJA225K010TNJ?qs=XLNwXgtzMM%2F9RK%2FJN7CZtw%3D%3D" H 750 1250 50  0001 L CNN "Mouser Price/Stock"
+F 8 "AVX" H 750 1150 50  0001 L CNN "Manufacturer_Name"
+F 9 "TAJA225K010TNJ" H 750 1050 50  0001 L CNN "Manufacturer_Part_Number"
+	1    650  1900
+	0    1    1    0
+$EndComp
+Wire Wire Line
+	1850 1800 1050 1800
+Wire Wire Line
+	850  1800 400  1800
+Wire Wire Line
+	750  1900 1850 1900
+$Comp
+L SamacSys_Parts:10k R8
+U 1 1 5F909097
+P 1100 1300
+F 0 "R8" V 875 1300 50  0000 C CNN
+F 1 "10k" V 966 1300 50  0000 C CNN
+F 2 "RESC1005X37N" H 1150 1150 50  0001 L CNN
+F 3 "https://componentsearchengine.com/Datasheets/1/MCS0402MC1002FE000.pdf" H 1150 1050 50  0001 L CNN
+F 4 "Thin Film Resistors - SMD .1W 10Kohms 1% 0402 50ppm Auto" H 1150 950 50  0001 L CNN "Description"
+F 5 "0.37" H 1150 850 50  0001 L CNN "Height"
+F 6 "594-MCS0402MC1002FE0" H 1150 750 50  0001 L CNN "Mouser Part Number"
+F 7 "https://www.mouser.com/Search/Refine.aspx?Keyword=594-MCS0402MC1002FE0" H 1150 650 50  0001 L CNN "Mouser Price/Stock"
+F 8 "Vishay" H 1150 550 50  0001 L CNN "Manufacturer_Name"
+F 9 "MCS0402MC1002FE000" H 1150 450 50  0001 L CNN "Manufacturer_Part_Number"
+	1    1100 1300
+	0    1    1    0
+$EndComp
+Wire Wire Line
+	1850 1400 1400 1400
+$Comp
+L SamacSys_Parts:10k R9
+U 1 1 5F90A7D1
+P 1300 1400
+F 0 "R9" V 1075 1400 50  0000 C CNN
+F 1 "10k" V 1166 1400 50  0000 C CNN
+F 2 "RESC1005X37N" H 1350 1250 50  0001 L CNN
+F 3 "https://componentsearchengine.com/Datasheets/1/MCS0402MC1002FE000.pdf" H 1350 1150 50  0001 L CNN
+F 4 "Thin Film Resistors - SMD .1W 10Kohms 1% 0402 50ppm Auto" H 1350 1050 50  0001 L CNN "Description"
+F 5 "0.37" H 1350 950 50  0001 L CNN "Height"
+F 6 "594-MCS0402MC1002FE0" H 1350 850 50  0001 L CNN "Mouser Part Number"
+F 7 "https://www.mouser.com/Search/Refine.aspx?Keyword=594-MCS0402MC1002FE0" H 1350 750 50  0001 L CNN "Mouser Price/Stock"
+F 8 "Vishay" H 1350 650 50  0001 L CNN "Manufacturer_Name"
+F 9 "MCS0402MC1002FE000" H 1350 550 50  0001 L CNN "Manufacturer_Part_Number"
+	1    1300 1400
+	0    1    1    0
+$EndComp
+$Comp
+L SamacSys_Parts:10k R10
+U 1 1 5F90AAEA
+P 1550 1600
+F 0 "R10" V 1325 1600 50  0000 C CNN
+F 1 "10k" V 1416 1600 50  0000 C CNN
+F 2 "RESC1005X37N" H 1600 1450 50  0001 L CNN
+F 3 "https://componentsearchengine.com/Datasheets/1/MCS0402MC1002FE000.pdf" H 1600 1350 50  0001 L CNN
+F 4 "Thin Film Resistors - SMD .1W 10Kohms 1% 0402 50ppm Auto" H 1600 1250 50  0001 L CNN "Description"
+F 5 "0.37" H 1600 1150 50  0001 L CNN "Height"
+F 6 "594-MCS0402MC1002FE0" H 1600 1050 50  0001 L CNN "Mouser Part Number"
+F 7 "https://www.mouser.com/Search/Refine.aspx?Keyword=594-MCS0402MC1002FE0" H 1600 950 50  0001 L CNN "Mouser Price/Stock"
+F 8 "Vishay" H 1600 850 50  0001 L CNN "Manufacturer_Name"
+F 9 "MCS0402MC1002FE000" H 1600 750 50  0001 L CNN "Manufacturer_Part_Number"
+	1    1550 1600
+	0    1    1    0
+$EndComp
+$Comp
+L SamacSys_Parts:100k R11
+U 1 1 5F921649
+P -1950 9750
+F 0 "R11" H -1891 9796 50  0000 L CNN
+F 1 "100k" H -1891 9705 50  0000 L CNN
+F 2 "RESC1005X40N" H -1900 9600 50  0001 L CNN
+F 3 "https://industrial.panasonic.com/cdbs/www-data/pdf/RDA0000/AOA0000C237.pdf" H -1900 9500 50  0001 L CNN
+F 4 "Panasonic ERA Series Thin Film Surface Mount Resistor 0402 Case 100k +/-0.5% 63mW +/-25ppm/C" H -1900 9400 50  0001 L CNN "Description"
+F 5 "0.4" H -1900 9300 50  0001 L CNN "Height"
+F 6 "667-ERA-2AED104X" H -1900 9200 50  0001 L CNN "Mouser Part Number"
+F 7 "https://www.mouser.co.uk/ProductDetail/Panasonic/ERA-2AED104X?qs=nho8PGNfA6oWiExMQMbJyw%3D%3D" H -1900 9100 50  0001 L CNN "Mouser Price/Stock"
+F 8 "Panasonic" H -1900 9000 50  0001 L CNN "Manufacturer_Name"
+F 9 "ERA-2AED104X" H -1900 8900 50  0001 L CNN "Manufacturer_Part_Number"
+	1    -1950 9750
+	1    0    0    -1
+$EndComp
