File: zx/pentagon 128 portable/schematic/Pentagon128 portable/stm32_power.sch (KiCad schematic (older format))
At the start: 40 parts

Commit message: updated schemes
Parts:
- gave numbers to parts that had none: 40

Commit message: updated BOM
Parts:
- removed C14, C19, C21: 1uF, Capacitor_SMD:C_0402_1005Metric, symbol Device:CP_Small
- removed C15, C20, C22, C23, C24, C25, C26, C27, C28, C29, C30, C31, C32, C33, C34, C35, C36, C37, C38, C39, C40, C41, C42, C43, C44, C45, C46, C47, C48, C49, C50, C51, C52: 100nF, Capacitor_SMD:C_0402_1005Metric, symbol Device:C_Small
- removed C16: 2.2uF, Capacitor_SMD:C_0402_1005Metric, symbol Device:C_Small
- removed C17, C18: 4.7uF, Capacitor_SMD:C_0402_1005Metric, symbol Device:CP_Small
- removed FB1: GZ2012D601TF, Capacitor_SMD:C_0805_2012Metric, symbol Device:Ferrite_Bead_Small
- added C14, C19, C21: 1uF, CAPC1005X33N, symbol SamacSys_Parts:1uF
- added C15, C20, C22, C23, C24, C25, C26, C27, C28, C29, C30, C31, C32, C33, C34, C35, C36, C37, C38, C39, C40, C41, C42, C43, C44, C45, C46, C47, C48, C49, C50, C51, C52: 100nF, CAPC1005X55N, symbol SamacSys_Parts:100nF
- added C16: 2.2uF, CAPC1005X55N, symbol SamacSys_Parts:2.2uF
- added C17, C18: 4.7uF, CAPC1005X55N, symbol SamacSys_Parts:4.7uF
- added FB1: BLM15PX601SZ1D, NFZ15SG152SN10B, symbol SamacSys_Parts:BLM15PX601SZ1D
